File: ampC.sch (KiCad schematic (older format))
At the start: 15 parts, among them U05 Mux, U07 TL084, U2 screw_term, U3 screw_term, U4 screw_term, U6 TL084

Commit message: added all adc outputs
Parts:
- renumbered R1 to R19, R2 to R20, R3 to R21, R4 to R22, R5 to R23, R6 to R24, R7 to R25, R8 to R26, R9 to R27, U05 to U010, U07 to U011, U6 to U12, U2 to U3, U4 to U9, U3 to U9

Commit message: added no connects on teensy
Parts:
- removed U010: Mux, Package_DIP:DIP-14_W7.62mm, symbol PNG_PCB_Parts:Mux
- removed U011: TL084, symbol PNG_PCB_Parts:Mux
Changed lines of the file:
@@
 AR Path="/6017DA21/6019D558" Ref="U?"  Part="1"
 AR Path="/601927EB/6019D558" Ref="U?"  Part="1"
-AR Path="/6019C043/6019D558" Ref="U010"  Part="1"
-AR Path="/601B4C16/6019D558" Ref="U021"  Part="1"
-F 0 "U021" H 3375 2515 50  0000 C CNN
+AR Path="/6019C043/6019D558" Ref="#U010"  Part="1"
+AR Path="/601B4C16/6019D558" Ref="#U021"  Part="1"
+F 0 "#U021" H 3375 2515 50  0000 C CNN
 F 1 "Mux" H 3375 2424 50  0000 C CNN
 F 2 "Package_DIP:DIP-14_W7.62mm" H 3350 2050 50  0001 C CNN
@@
 AR Path="/6017CC5E/6019D562" Ref="U?"  Part="3"
 AR Path="/601927EB/6019D562" Ref="U?"  Part="3"
-AR Path="/6019C043/6019D562" Ref="U011"  Part="3"
-AR Path="/601B4C16/6019D562" Ref="U022"  Part="3"
-F 0 "U022" H 5928 2221 50  0000 L CNN
+AR Path="/6019C043/6019D562" Ref="#U011"  Part="3"
+AR Path="/601B4C16/6019D562" Ref="#U022"  Part="3"
+F 0 "#U022" H 5928 2221 50  0000 L CNN
 F 1 "TL084" H 5928 2130 50  0000 L CNN
 F 2 "" H 5700 2100 50  0001 C CNN

Commit message: added footprint to some op amps
Parts:
- U12: footprint (none) -> Package_DIP:DIP-14_W7.62mm
Changed lines of the file:
@@
 $Descr A4 11693 8268
 encoding utf-8
-Sheet 8 11
+Sheet 4 11
 Title ""
 Date ""
@@
 AR Path="/6019C043/6019D554" Ref="#PWR024"  Part="1"
 AR Path="/601B4C16/6019D554" Ref="#PWR054"  Part="1"
-F 0 "#PWR054" H 1450 1850 50  0001 C CNN
+F 0 "#PWR024" H 1450 1850 50  0001 C CNN
 F 1 "GND" H 1455 1927 50  0000 C CNN
 F 2 "" H 1450 2100 50  0001 C CNN
@@
 AR Path="/6019C043/6019D566" Ref="U12"  Part="3"
 AR Path="/601B4C16/6019D566" Ref="U7"  Part="3"
-F 0 "U7" H 6000 3433 50  0000 C CNN
+F 0 "U12" H 6000 3433 50  0000 C CNN
 F 1 "TL084" H 6000 3524 50  0000 C CNN
-F 2 "" H 5950 3900 50  0001 C CNN
+F 2 "Package_DIP:DIP-14_W7.62mm" H 5950 3900 50  0001 C CNN
 F 3 "http://www.ti.com/lit/ds/symlink/tl081.pdf" H 6050 4000 50  0001 C CNN
 	3    6000 3800
@@
 AR Path="/6019C043/60198F28" Ref="R26"  Part="1"
 AR Path="/601B4C16/60198F28" Ref="R62"  Part="1"
-F 0 "R62" H 5520 4096 50  0000 L CNN
+F 0 "R26" H 5520 4096 50  0000 L CNN
 F 1 "15" H 5520 4005 50  0000 L CNN
 F 2 "Resistor_THT:R_Axial_DIN0204_L3.6mm_D1.6mm_P5.08mm_Horizontal" V 5380 4050 50  0001 C CNN
@@
 AR Path="/6019C043/6019D567" Ref="R27"  Part="1"
 AR Path="/601B4C16/6019D567" Ref="R63"  Part="1"
-F 0 "R63" V 5743 3250 50  0000 C CNN
+F 0 "R27" V 5743 3250 50  0000 C CNN
 F 1 "15" V 5834 3250 50  0000 C CNN
 F 2 "Resistor_THT:R_Axial_DIN0204_L3.6mm_D1.6mm_P5.08mm_Horizontal" V 5880 3250 50  0001 C CNN
@@
 AR Path="/6019C043/6019D55D" Ref="R24"  Part="1"
 AR Path="/601B4C16/6019D55D" Ref="R60"  Part="1"
-F 0 "R60" V 5307 3700 50  0000 C CNN
+F 0 "R24" V 5307 3700 50  0000 C CNN
 F 1 "1" V 5216 3700 50  0000 C CNN
 F 2 "Resistor_THT:R_Axial_DIN0204_L3.6mm_D1.6mm_P5.08mm_Horizontal" V 5030 3700 50  0001 C CNN
@@
 AR Path="/6019C043/60198F34" Ref="R25"  Part="1"
 AR Path="/601B4C16/60198F34" Ref="R61"  Part="1"
-F 0 "R61" V 5000 3900 50  0000 C CNN
+F 0 "R25" V 5000 3900 50  0000 C CNN
 F 1 "1" V 4900 3900 50  0000 C CNN
 F 2 "Resistor_THT:R_Axial_DIN0204_L3.6mm_D1.6mm_P5.08mm_Horizontal" V 5030 3900 50  0001 C CNN
@@
 AR Path="/6019C043/6017E433" Ref="R22"  Part="1"
 AR Path="/601B4C16/6017E433" Ref="R58"  Part="1"
-F 0 "R58" H 3320 3546 50  0000 L CNN
+F 0 "R22" H 3320 3546 50  0000 L CNN
 F 1 "330" H 3320 3455 50  0000 L CNN
 F 2 "Resistor_THT:R_Axial_DIN0204_L3.6mm_D1.6mm_P5.08mm_Horizontal" V 3180 3500 50  0001 C CNN
@@
 AR Path="/6019C043/6017E434" Ref="R23"  Part="1"
 AR Path="/601B4C16/6017E434" Ref="R59"  Part="1"
-F 0 "R59" H 3320 3846 50  0000 L CNN
+F 0 "R23" H 3320 3846 50  0000 L CNN
 F 1 "560" H 3320 3755 50  0000 L CNN
 F 2 "Resistor_THT:R_Axial_DIN0204_L3.6mm_D1.6mm_P5.08mm_Horizontal" V 3180 3800 50  0001 C CNN
@@
 AR Path="/6019C043/6017E435" Ref="#PWR027"  Part="1"
 AR Path="/601B4C16/6017E435" Ref="#PWR057"  Part="1"
-F 0 "#PWR057" H 3250 3200 50  0001 C CNN
+F 0 "#PWR027" H 3250 3200 50  0001 C CNN
 F 1 "+3.3V" H 3265 3523 50  0000 C CNN
 F 2 "" H 3250 3350 50  0001 C CNN
@@
 AR Path="/6019C043/6019D569" Ref="#PWR028"  Part="1"
 AR Path="/601B4C16/6019D569" Ref="#PWR058"  Part="1"
-F 0 "#PWR058" H 3250 3700 50  0001 C CNN
+F 0 "#PWR028" H 3250 3700 50  0001 C CNN
 F 1 "GND" H 3255 3777 50  0000 C CNN
 F 2 "" H 3250 3950 50  0001 C CNN
@@
 AR Path="/6019C043/6019D555" Ref="#PWR029"  Part="1"
 AR Path="/601B4C16/6019D555" Ref="#PWR059"  Part="1"
-F 0 "#PWR059" H 5450 3950 50  0001 C CNN
+F 0 "#PWR029" H 5450 3950 50  0001 C CNN
 F 1 "GND" H 5455 4027 50  0000 C CNN
 F 2 "" H 5450 4200 50  0001 C CNN
@@
 AR Path="/6019C043/6019D556" Ref="R19"  Part="1"
 AR Path="/601B4C16/6019D556" Ref="R55"  Part="1"
-F 0 "R55" H 1520 1996 50  0000 L CNN
+F 0 "R19" H 1520 1996 50  0000 L CNN
 F 1 "330" H 1520 1905 50  0000 L CNN
 F 2 "Resistor_THT:R_Axial_DIN0204_L3.6mm_D1.6mm_P5.08mm_Horizontal" V 1380 1950 50  0001 C CNN
@@
 AR Path="/6019C043/6019D558" Ref="#U010"  Part="1"
 AR Path="/601B4C16/6019D558" Ref="#U021"  Part="1"
-F 0 "#U021" H 3375 2515 50  0000 C CNN
+F 0 "#U010" H 3375 2515 50  0000 C CNN
 F 1 "Mux" H 3375 2424 50  0000 C CNN
 F 2 "Package_DIP:DIP-14_W7.62mm" H 3350 2050 50  0001 C CNN
@@
 AR Path="/6019C043/6019D557" Ref="U3"  Part="1"
 AR Path="/601B4C16/6019D557" Ref="U19"  Part="1"
-F 0 "U19" H 1508 1934 50  0000 L CNN
+F 0 "U3" H 1508 1934 50  0000 L CNN
 F 1 "screw_term" H 1508 1843 50  0000 L CNN
 F 2 "Connector_PinHeader_1.27mm:PinHeader_1x02_P1.27mm_Vertical" H 1450 1800 50  0001 C CNN
@@
 AR Path="/6019C043/60176F19" Ref="#PWR025"  Part="1"
 AR Path="/601B4C16/60176F19" Ref="#PWR055"  Part="1"
-F 0 "#PWR055" H 1450 2800 50  0001 C CNN
+F 0 "#PWR025" H 1450 2800 50  0001 C CNN
 F 1 "GND" H 1455 2877 50  0000 C CNN
 F 2 "" H 1450 3050 50  0001 C CNN
@@
 AR Path="/6019C043/60198F39" Ref="R20"  Part="1"
 AR Path="/601B4C16/60198F39" Ref="R56"  Part="1"
-F 0 "R56" H 1520 2946 50  0000 L CNN
+F 0 "R20" H 1520 2946 50  0000 L CNN
 F 1 "330" H 1520 2855 50  0000 L CNN
 F 2 "Resistor_THT:R_Axial_DIN0204_L3.6mm_D1.6mm_P5.08mm_Horizontal" V 1380 2900 50  0001 C CNN
@@
 AR Path="/6019C043/6019D55A" Ref="U9"  Part="2"
 AR Path="/601B4C16/6019D55A" Ref="U20"  Part="2"
-F 0 "U20" H 1508 2884 50  0000 L CNN
+F 0 "U9" H 1508 2884 50  0000 L CNN
 F 1 "screw_term" H 1508 2793 50  0000 L CNN
 F 2 "Connector_PinHeader_1.27mm:PinHeader_1x02_P1.27mm_Vertical" H 1450 2750 50  0001 C CNN
@@
 AR Path="/6019C043/60177983" Ref="#PWR026"  Part="1"
 AR Path="/601B4C16/60177983" Ref="#PWR056"  Part="1"
-F 0 "#PWR056" H 1450 3800 50  0001 C CNN
+F 0 "#PWR026" H 1450 3800 50  0001 C CNN
 F 1 "GND" H 1455 3877 50  0000 C CNN
 F 2 "" H 1450 4050 50  0001 C CNN
@@
 AR Path="/6019C043/6019D561" Ref="R21"  Part="1"
 AR Path="/601B4C16/6019D561" Ref="R57"  Part="1"
-F 0 "R57" H 1520 3946 50  0000 L CNN
+F 0 "R21" H 1520 3946 50  0000 L CNN
 F 1 "330" H 1520 3855 50  0000 L CNN
 F 2 "Resistor_THT:R_Axial_DIN0204_L3.6mm_D1.6mm_P5.08mm_Horizontal" V 1380 3900 50  0001 C CNN
@@
 AR Path="/6019C043/6017798F" Ref="U9"  Part="1"
 AR Path="/601B4C16/6017798F" Ref="U20"  Part="1"
-F 0 "U20" H 1508 3884 50  0000 L CNN
+F 0 "U9" H 1508 3884 50  0000 L CNN
 F 1 "screw_term" H 1508 3793 50  0000 L CNN
 F 2 "Connector_PinHeader_1.27mm:PinHeader_1x02_P1.27mm_Vertical" H 1450 3750 50  0001 C CNN
@@
 AR Path="/6019C043/6019D562" Ref="#U011"  Part="3"
 AR Path="/601B4C16/6019D562" Ref="#U022"  Part="3"
-F 0 "#U022" H 5928 2221 50  0000 L CNN
+F 0 "#U011" H 5928 2221 50  0000 L CNN
 F 1 "TL084" H 5928 2130 50  0000 L CNN
 F 2 "" H 5700 2100 50  0001 C CNN
@@
 AR Path="/6019C043/6019D563" Ref="#PWR031"  Part="1"
 AR Path="/601B4C16/6019D563" Ref="#PWR061"  Part="1"
-F 0 "#PWR061" H 5700 2050 50  0001 C CNN
+F 0 "#PWR031" H 5700 2050 50  0001 C CNN
 F 1 "GND" H 5705 2127 50  0000 C CNN
 F 2 "" H 5700 2300 50  0001 C CNN
@@
 AR Path="/6019C043/6019D564" Ref="#PWR030"  Part="1"
 AR Path="/601B4C16/6019D564" Ref="#PWR060"  Part="1"
-F 0 "#PWR060" H 5700 1600 50  0001 C CNN
+F 0 "#PWR030" H 5700 1600 50  0001 C CNN
 F 1 "+3.3V" H 5715 1923 50  0000 C CNN
 F 2 "" H 5700 1750 50  0001 C CNN

Commit message: updated all mux packages in eeschema
Changed lines of the file:
@@
 $Descr A4 11693 8268
 encoding utf-8
-Sheet 4 11
+Sheet 8 11
 Title ""
 Date ""
@@
 AR Path="/6019C043/6019D554" Ref="#PWR024"  Part="1"
 AR Path="/601B4C16/6019D554" Ref="#PWR054"  Part="1"
-F 0 "#PWR024" H 1450 1850 50  0001 C CNN
+F 0 "#PWR054" H 1450 1850 50  0001 C CNN
 F 1 "GND" H 1455 1927 50  0000 C CNN
 F 2 "" H 1450 2100 50  0001 C CNN
@@
 AR Path="/6019C043/6019D566" Ref="U12"  Part="3"
 AR Path="/601B4C16/6019D566" Ref="U7"  Part="3"
-F 0 "U12" H 6000 3433 50  0000 C CNN
+F 0 "U7" H 6000 3433 50  0000 C CNN
 F 1 "TL084" H 6000 3524 50  0000 C CNN
 F 2 "Package_DIP:DIP-14_W7.62mm" H 5950 3900 50  0001 C CNN
@@
 AR Path="/6019C043/60198F28" Ref="R26"  Part="1"
 AR Path="/601B4C16/60198F28" Ref="R62"  Part="1"
-F 0 "R26" H 5520 4096 50  0000 L CNN
+F 0 "R62" H 5520 4096 50  0000 L CNN
 F 1 "15" H 5520 4005 50  0000 L CNN
 F 2 "Resistor_THT:R_Axial_DIN0204_L3.6mm_D1.6mm_P5.08mm_Horizontal" V 5380 4050 50  0001 C CNN
@@
 AR Path="/6019C043/6019D567" Ref="R27"  Part="1"
 AR Path="/601B4C16/6019D567" Ref="R63"  Part="1"
-F 0 "R27" V 5743 3250 50  0000 C CNN
+F 0 "R63" V 5743 3250 50  0000 C CNN
 F 1 "15" V 5834 3250 50  0000 C CNN
 F 2 "Resistor_THT:R_Axial_DIN0204_L3.6mm_D1.6mm_P5.08mm_Horizontal" V 5880 3250 50  0001 C CNN
@@
 AR Path="/6019C043/6019D55D" Ref="R24"  Part="1"
 AR Path="/601B4C16/6019D55D" Ref="R60"  Part="1"
-F 0 "R24" V 5307 3700 50  0000 C CNN
+F 0 "R60" V 5307 3700 50  0000 C CNN
 F 1 "1" V 5216 3700 50  0000 C CNN
 F 2 "Resistor_THT:R_Axial_DIN0204_L3.6mm_D1.6mm_P5.08mm_Horizontal" V 5030 3700 50  0001 C CNN
@@
 AR Path="/6019C043/60198F34" Ref="R25"  Part="1"
 AR Path="/601B4C16/60198F34" Ref="R61"  Part="1"
-F 0 "R25" V 5000 3900 50  0000 C CNN
+F 0 "R61" V 5000 3900 50  0000 C CNN
 F 1 "1" V 4900 3900 50  0000 C CNN
 F 2 "Resistor_THT:R_Axial_DIN0204_L3.6mm_D1.6mm_P5.08mm_Horizontal" V 5030 3900 50  0001 C CNN
@@
 AR Path="/6019C043/6017E433" Ref="R22"  Part="1"
 AR Path="/601B4C16/6017E433" Ref="R58"  Part="1"
-F 0 "R22" H 3320 3546 50  0000 L CNN
+F 0 "R58" H 3320 3546 50  0000 L CNN
 F 1 "330" H 3320 3455 50  0000 L CNN
 F 2 "Resistor_THT:R_Axial_DIN0204_L3.6mm_D1.6mm_P5.08mm_Horizontal" V 3180 3500 50  0001 C CNN
@@
 AR Path="/6019C043/6017E434" Ref="R23"  Part="1"
 AR Path="/601B4C16/6017E434" Ref="R59"  Part="1"
-F 0 "R23" H 3320 3846 50  0000 L CNN
+F 0 "R59" H 3320 3846 50  0000 L CNN
 F 1 "560" H 3320 3755 50  0000 L CNN
 F 2 "Resistor_THT:R_Axial_DIN0204_L3.6mm_D1.6mm_P5.08mm_Horizontal" V 3180 3800 50  0001 C CNN
@@
 AR Path="/6019C043/6017E435" Ref="#PWR027"  Part="1"
 AR Path="/601B4C16/6017E435" Ref="#PWR057"  Part="1"
-F 0 "#PWR027" H 3250 3200 50  0001 C CNN
+F 0 "#PWR057" H 3250 3200 50  0001 C CNN
 F 1 "+3.3V" H 3265 3523 50  0000 C CNN
 F 2 "" H 3250 3350 50  0001 C CNN
@@
 AR Path="/6019C043/6019D569" Ref="#PWR028"  Part="1"
 AR Path="/601B4C16/6019D569" Ref="#PWR058"  Part="1"
-F 0 "#PWR028" H 3250 3700 50  0001 C CNN
+F 0 "#PWR058" H 3250 3700 50  0001 C CNN
 F 1 "GND" H 3255 3777 50  0000 C CNN
 F 2 "" H 3250 3950 50  0001 C CNN
@@
 AR Path="/6019C043/6019D555" Ref="#PWR029"  Part="1"
 AR Path="/601B4C16/6019D555" Ref="#PWR059"  Part="1"
-F 0 "#PWR029" H 5450 3950 50  0001 C CNN
+F 0 "#PWR059" H 5450 3950 50  0001 C CNN
 F 1 "GND" H 5455 4027 50  0000 C CNN
 F 2 "" H 5450 4200 50  0001 C CNN
@@
 AR Path="/6019C043/6019D556" Ref="R19"  Part="1"
 AR Path="/601B4C16/6019D556" Ref="R55"  Part="1"
-F 0 "R19" H 1520 1996 50  0000 L CNN
+F 0 "R55" H 1520 1996 50  0000 L CNN
 F 1 "330" H 1520 1905 50  0000 L CNN
 F 2 "Resistor_THT:R_Axial_DIN0204_L3.6mm_D1.6mm_P5.08mm_Horizontal" V 1380 1950 50  0001 C CNN
@@
 AR Path="/6019C043/6019D558" Ref="#U010"  Part="1"
 AR Path="/601B4C16/6019D558" Ref="#U021"  Part="1"
-F 0 "#U010" H 3375 2515 50  0000 C CNN
+F 0 "#U021" H 3375 2515 50  0000 C CNN
 F 1 "Mux" H 3375 2424 50  0000 C CNN
-F 2 "Package_DIP:DIP-14_W7.62mm" H 3350 2050 50  0001 C CNN
+F 2 "Package_DIP:DIP-16_W7.62mm" H 3350 2050 50  0001 C CNN
 F 3 "" H 3350 2050 50  0001 C CNN
 	1    3350 2050
@@
 AR Path="/6019C043/6019D557" Ref="U3"  Part="1"
 AR Path="/601B4C16/6019D557" Ref="U19"  Part="1"
-F 0 "U3" H 1508 1934 50  0000 L CNN
+F 0 "U19" H 1508 1934 50  0000 L CNN
 F 1 "screw_term" H 1508 1843 50  0000 L CNN
 F 2 "Connector_PinHeader_1.27mm:PinHeader_1x02_P1.27mm_Vertical" H 1450 1800 50  0001 C CNN
@@
 AR Path="/6019C043/60176F19" Ref="#PWR025"  Part="1"
 AR Path="/601B4C16/60176F19" Ref="#PWR055"  Part="1"
-F 0 "#PWR025" H 1450 2800 50  0001 C CNN
+F 0 "#PWR055" H 1450 2800 50  0001 C CNN
 F 1 "GND" H 1455 2877 50  0000 C CNN
 F 2 "" H 1450 3050 50  0001 C CNN
@@
 AR Path="/6019C043/60198F39" Ref="R20"  Part="1"
 AR Path="/601B4C16/60198F39" Ref="R56"  Part="1"
-F 0 "R20" H 1520 2946 50  0000 L CNN
+F 0 "R56" H 1520 2946 50  0000 L CNN
 F 1 "330" H 1520 2855 50  0000 L CNN
 F 2 "Resistor_THT:R_Axial_DIN0204_L3.6mm_D1.6mm_P5.08mm_Horizontal" V 1380 2900 50  0001 C CNN
@@
 AR Path="/6019C043/6019D55A" Ref="U9"  Part="2"
 AR Path="/601B4C16/6019D55A" Ref="U20"  Part="2"
-F 0 "U9" H 1508 2884 50  0000 L CNN
+F 0 "U20" H 1508 2884 50  0000 L CNN
 F 1 "screw_term" H 1508 2793 50  0000 L CNN
 F 2 "Connector_PinHeader_1.27mm:PinHeader_1x02_P1.27mm_Vertical" H 1450 2750 50  0001 C CNN
@@
 AR Path="/6019C043/60177983" Ref="#PWR026"  Part="1"
 AR Path="/601B4C16/60177983" Ref="#PWR056"  Part="1"
-F 0 "#PWR026" H 1450 3800 50  0001 C CNN
+F 0 "#PWR056" H 1450 3800 50  0001 C CNN
 F 1 "GND" H 1455 3877 50  0000 C CNN
 F 2 "" H 1450 4050 50  0001 C CNN
@@
 AR Path="/6019C043/6019D561" Ref="R21"  Part="1"
 AR Path="/601B4C16/6019D561" Ref="R57"  Part="1"
-F 0 "R21" H 1520 3946 50  0000 L CNN
+F 0 "R57" H 1520 3946 50  0000 L CNN
 F 1 "330" H 1520 3855 50  0000 L CNN
 F 2 "Resistor_THT:R_Axial_DIN0204_L3.6mm_D1.6mm_P5.08mm_Horizontal" V 1380 3900 50  0001 C CNN
@@
 AR Path="/6019C043/6017798F" Ref="U9"  Part="1"
 AR Path="/601B4C16/6017798F" Ref="U20"  Part="1"
-F 0 "U9" H 1508 3884 50  0000 L CNN
+F 0 "U20" H 1508 3884 50  0000 L CNN
 F 1 "screw_term" H 1508 3793 50  0000 L CNN
 F 2 "Connector_PinHeader_1.27mm:PinHeader_1x02_P1.27mm_Vertical" H 1450 3750 50  0001 C CNN
@@
 AR Path="/6019C043/6019D562" Ref="#U011"  Part="3"
 AR Path="/601B4C16/6019D562" Ref="#U022"  Part="3"
-F 0 "#U011" H 5928 2221 50  0000 L CNN
+F 0 "#U022" H 5928 2221 50  0000 L CNN
 F 1 "TL084" H 5928 2130 50  0000 L CNN
 F 2 "" H 5700 2100 50  0001 C CNN
@@
 AR Path="/6019C043/6019D563" Ref="#PWR031"  Part="1"
 AR Path="/601B4C16/6019D563" Ref="#PWR061"  Part="1"
-F 0 "#PWR031" H 5700 2050 50  0001 C CNN
+F 0 "#PWR061" H 5700 2050 50  0001 C CNN
 F 1 "GND" H 5705 2127 50  0000 C CNN
 F 2 "" H 5700 2300 50  0001 C CNN
@@
 AR Path="/6019C043/6019D564" Ref="#PWR030"  Part="1"
 AR Path="/601B4C16/6019D564" Ref="#PWR060"  Part="1"
-F 0 "#PWR030" H 5700 1600 50  0001 C CNN
+F 0 "#PWR060" H 5700 1600 50  0001 C CNN
 F 1 "+3.3V" H 5715 1923 50  0000 C CNN
 F 2 "" H 5700 1750 50  0001 C CNN

Commit message: added all muxes to the board
Parts:
- added U19: Mux, Package_DIP:DIP-16_W7.62mm, symbol PNG_PCB_Parts:Mux
- renumbered U12 to U6, U3 to U8, U9 to U8
Connections:
- net +3V3: now also U19.16 (Vdd)
- net GND: now also U19.6 (INH), U19.7 (VEE), U19.8 (Vss)
- net V1: now also U19.13 (xout)
- net mux0: now also U19.12 (x0)
- net mux1: now also U19.14 (x1)
- net mux2: now also U19.15 (x2)
- net selA: now also U19.10 (selA)
- net selB: now also U19.9 (selB)
Changed lines of the file:
@@
 AR Path="/6017DA21/6019D566" Ref="U?"  Part="1"
 AR Path="/601927EB/6019D566" Ref="U?"  Part="1"
-AR Path="/6019C043/6019D566" Ref="U12"  Part="3"
-AR Path="/601B4C16/6019D566" Ref="U7"  Part="3"
-F 0 "U7" H 6000 3433 50  0000 C CNN
+AR Path="/6019C043/6019D566" Ref="U6"  Part="3"
+AR Path="/601B4C16/6019D566" Ref="U15"  Part="3"
+F 0 "U15" H 6000 3433 50  0000 C CNN
 F 1 "TL084" H 6000 3524 50  0000 C CNN
 F 2 "Package_DIP:DIP-14_W7.62mm" H 5950 3900 50  0001 C CNN
@@
 $EndComp
 $Comp
-L PNG_PCB_Parts:Mux U?
-U 1 1 6019D558
-P 3350 2050
-AR Path="/60132BC3/6013AE22/6019D558" Ref="U?"  Part="1"
-AR Path="/6017CC5E/6019D558" Ref="U?"  Part="1"
-AR Path="/6017DA21/6019D558" Ref="U?"  Part="1"
-AR Path="/601927EB/6019D558" Ref="U?"  Part="1"
-AR Path="/6019C043/6019D558" Ref="#U010"  Part="1"
-AR Path="/601B4C16/6019D558" Ref="#U021"  Part="1"
-F 0 "#U021" H 3375 2515 50  0000 C CNN
-F 1 "Mux" H 3375 2424 50  0000 C CNN
-F 2 "Package_DIP:DIP-16_W7.62mm" H 3350 2050 50  0001 C CNN
-F 3 "" H 3350 2050 50  0001 C CNN
-	1    3350 2050
-	1    0    0    -1
-$EndComp
-$Comp
 L PNG_PCB_Parts:screw_term U?
 U 1 1 6019D557
@@
 AR Path="/6017DA21/6019D557" Ref="U?"  Part="1"
 AR Path="/601927EB/6019D557" Ref="U?"  Part="1"
-AR Path="/6019C043/6019D557" Ref="U3"  Part="1"
-AR Path="/601B4C16/6019D557" Ref="U19"  Part="1"
-F 0 "U19" H 1508 1934 50  0000 L CNN
+AR Path="/6019C043/6019D557" Ref="U8"  Part="1"
+AR Path="/601B4C16/6019D557" Ref="U17"  Part="1"
+F 0 "U17" H 1508 1934 50  0000 L CNN
 F 1 "screw_term" H 1508 1843 50  0000 L CNN
 F 2 "Connector_PinHeader_1.27mm:PinHeader_1x02_P1.27mm_Vertical" H 1450 1800 50  0001 C CNN
@@
 AR Path="/6017DA21/6019D55A" Ref="U?"  Part="1"
 AR Path="/601927EB/6019D55A" Ref="U?"  Part="2"
-AR Path="/6019C043/6019D55A" Ref="U9"  Part="2"
-AR Path="/601B4C16/6019D55A" Ref="U20"  Part="2"
-F 0 "U20" H 1508 2884 50  0000 L CNN
+AR Path="/6019C043/6019D55A" Ref="U8"  Part="2"
+AR Path="/601B4C16/6019D55A" Ref="U17"  Part="2"
+F 0 "U17" H 1508 2884 50  0000 L CNN
 F 1 "screw_term" H 1508 2793 50  0000 L CNN
 F 2 "Connector_PinHeader_1.27mm:PinHeader_1x02_P1.27mm_Vertical" H 1450 2750 50  0001 C CNN
@@
 AR Path="/601927EB/6017798F" Ref="U?"  Part="1"
 AR Path="/6019C043/6017798F" Ref="U9"  Part="1"
-AR Path="/601B4C16/6017798F" Ref="U20"  Part="1"
-F 0 "U20" H 1508 3884 50  0000 L CNN
+AR Path="/601B4C16/6017798F" Ref="U18"  Part="1"
+F 0 "U18" H 1508 3884 50  0000 L CNN
 F 1 "screw_term" H 1508 3793 50  0000 L CNN
 F 2 "Connector_PinHeader_1.27mm:PinHeader_1x02_P1.27mm_Vertical" H 1450 3750 50  0001 C CNN
@@
 Text Label 2700 2150 0    50   ~ 0
 mux2
-$Comp
-L PNG_PCB_Parts:Mux U?
-U 3 1 6019D562
-P 5700 2100
-AR Path="/6017CC5E/6019D562" Ref="U?"  Part="3"
-AR Path="/601927EB/6019D562" Ref="U?"  Part="3"
-AR Path="/6019C043/6019D562" Ref="#U011"  Part="3"
-AR Path="/601B4C16/6019D562" Ref="#U022"  Part="3"
-F 0 "#U022" H 5928 2221 50  0000 L CNN
-F 1 "TL084" H 5928 2130 50  0000 L CNN
-F 2 "" H 5700 2100 50  0001 C CNN
-F 3 "http://www.ti.com/lit/ds/symlink/tl081.pdf" H 5700 2100 50  0001 C CNN
-	3    5700 2100
-	1    0    0    -1
-$EndComp
 Wire Wire Line
 	5600 2300 5700 2300
@@
 Text HLabel 5200 2050 0    50   Input ~ 0
 selB
+$Comp
+L PNG_PCB_Parts:Mux U19
+U 1 1 601763C1
+P 3350 2050
+AR Path="/601B4C16/601763C1" Ref="U19"  Part="1"
+AR Path="/6019C043/601763C1" Ref="U10"  Part="1"
+F 0 "U19" H 3375 2515 50  0000 C CNN
+F 1 "Mux" H 3375 2424 50  0000 C CNN
+F 2 "Package_DIP:DIP-16_W7.62mm" H 3350 2050 50  0001 C CNN
+F 3 "" H 3350 2050 50  0001 C CNN
+	1    3350 2050
+	1    0    0    -1
+$EndComp
+$Comp
+L PNG_PCB_Parts:Mux U19
+U 3 1 60176BAF
+P 5700 2100
+AR Path="/601B4C16/60176BAF" Ref="U19"  Part="3"
+AR Path="/6019C043/60176BAF" Ref="U10"  Part="3"
+F 0 "U19" H 5928 2221 50  0000 L CNN
+F 1 "Mux" H 5928 2130 50  0000 L CNN
+F 2 "Package_DIP:DIP-16_W7.62mm" H 5700 2100 50  0001 C CNN
+F 3 "" H 5700 2100 50  0001 C CNN
+	3    5700 2100
+	1    0    0    -1
+$EndComp
 $EndSCHEMATC
