File: ampD.sch (KiCad schematic (older format))
At the start: 14 parts, among them U05 Mux, U2 screw_term, U3 screw_term, U4 screw_term, U6 TL084

Commit message: added all adc outputs
Parts:
- renumbered R1 to R28, R2 to R29, R3 to R30, R4 to R31, R5 to R32, R6 to R33, R7 to R34, R8 to R35, R9 to R36, U05 to U010, U6 to U12, U3 to U13, U2 to U13, U4 to U14

Commit message: added no connects on teensy
Parts:
- removed U010: Mux, symbol PNG_PCB_Parts:Mux
Changed lines of the file:
@@
 AR Path="/601927EB/60198F2C" Ref="U?"  Part="2"
 AR Path="/6019DBCE/60198F2C" Ref="U?"  Part="2"
-AR Path="/6019DBCE/6019E3AE" Ref="U010"  Part="2"
-AR Path="/601B4C19/6019E3AE" Ref="U021"  Part="2"
-F 0 "U021" H 3375 2515 50  0000 C CNN
+AR Path="/6019DBCE/6019E3AE" Ref="#U010"  Part="2"
+AR Path="/601B4C19/6019E3AE" Ref="#U021"  Part="2"
+F 0 "#U021" H 3375 2515 50  0000 C CNN
 F 1 "Mux" H 3375 2424 50  0000 C CNN
 F 2 "" H 3350 2050 50  0001 C CNN

Commit message: added footprint to some op amps
Parts:
- U12: footprint (none) -> Package_DIP:DIP-14_W7.62mm
Changed lines of the file:
@@
 AR Path="/6019DBCE/60198F27" Ref="#PWR032"  Part="1"
 AR Path="/601B4C19/60198F27" Ref="#PWR062"  Part="1"
-F 0 "#PWR062" H 1450 1850 50  0001 C CNN
+F 0 "#PWR032" H 1450 1850 50  0001 C CNN
 F 1 "GND" H 1455 1927 50  0000 C CNN
 F 2 "" H 1450 2100 50  0001 C CNN
@@
 AR Path="/6019DBCE/6015EF5C" Ref="R35"  Part="1"
 AR Path="/601B4C19/6015EF5C" Ref="R71"  Part="1"
-F 0 "R71" H 5520 4096 50  0000 L CNN
+F 0 "R35" H 5520 4096 50  0000 L CNN
 F 1 "15" H 5520 4005 50  0000 L CNN
 F 2 "Resistor_THT:R_Axial_DIN0204_L3.6mm_D1.6mm_P5.08mm_Horizontal" V 5380 4050 50  0001 C CNN
@@
 AR Path="/6019DBCE/6019E3A7" Ref="R36"  Part="1"
 AR Path="/601B4C19/6019E3A7" Ref="R72"  Part="1"
-F 0 "R72" V 5743 3250 50  0000 C CNN
+F 0 "R36" V 5743 3250 50  0000 C CNN
 F 1 "15" V 5834 3250 50  0000 C CNN
 F 2 "Resistor_THT:R_Axial_DIN0204_L3.6mm_D1.6mm_P5.08mm_Horizontal" V 5880 3250 50  0001 C CNN
@@
 AR Path="/6019DBCE/6019E3B2" Ref="R33"  Part="1"
 AR Path="/601B4C19/6019E3B2" Ref="R69"  Part="1"
-F 0 "R69" V 5307 3700 50  0000 C CNN
+F 0 "R33" V 5307 3700 50  0000 C CNN
 F 1 "1" V 5216 3700 50  0000 C CNN
 F 2 "Resistor_THT:R_Axial_DIN0204_L3.6mm_D1.6mm_P5.08mm_Horizontal" V 5030 3700 50  0001 C CNN
@@
 AR Path="/6019DBCE/6019E3A8" Ref="R34"  Part="1"
 AR Path="/601B4C19/6019E3A8" Ref="R70"  Part="1"
-F 0 "R70" V 5000 3900 50  0000 C CNN
+F 0 "R34" V 5000 3900 50  0000 C CNN
 F 1 "1" V 4900 3900 50  0000 C CNN
 F 2 "Resistor_THT:R_Axial_DIN0204_L3.6mm_D1.6mm_P5.08mm_Horizontal" V 5030 3900 50  0001 C CNN
@@
 AR Path="/6019DBCE/6019E3B3" Ref="R31"  Part="1"
 AR Path="/601B4C19/6019E3B3" Ref="R67"  Part="1"
-F 0 "R67" H 3320 3546 50  0000 L CNN
+F 0 "R31" H 3320 3546 50  0000 L CNN
 F 1 "330" H 3320 3455 50  0000 L CNN
 F 2 "Resistor_THT:R_Axial_DIN0204_L3.6mm_D1.6mm_P5.08mm_Horizontal" V 3180 3500 50  0001 C CNN
@@
 AR Path="/6019DBCE/60198F36" Ref="R32"  Part="1"
 AR Path="/601B4C19/60198F36" Ref="R68"  Part="1"
-F 0 "R68" H 3320 3846 50  0000 L CNN
+F 0 "R32" H 3320 3846 50  0000 L CNN
 F 1 "560" H 3320 3755 50  0000 L CNN
 F 2 "Resistor_THT:R_Axial_DIN0204_L3.6mm_D1.6mm_P5.08mm_Horizontal" V 3180 3800 50  0001 C CNN
@@
 AR Path="/6019DBCE/60198F37" Ref="#PWR035"  Part="1"
 AR Path="/601B4C19/60198F37" Ref="#PWR065"  Part="1"
-F 0 "#PWR065" H 3250 3200 50  0001 C CNN
+F 0 "#PWR035" H 3250 3200 50  0001 C CNN
 F 1 "+3.3V" H 3265 3523 50  0000 C CNN
 F 2 "" H 3250 3350 50  0001 C CNN
@@
 AR Path="/6019DBCE/6019E3A9" Ref="#PWR036"  Part="1"
 AR Path="/601B4C19/6019E3A9" Ref="#PWR066"  Part="1"
-F 0 "#PWR066" H 3250 3700 50  0001 C CNN
+F 0 "#PWR036" H 3250 3700 50  0001 C CNN
 F 1 "GND" H 3255 3777 50  0000 C CNN
 F 2 "" H 3250 3950 50  0001 C CNN
@@
 AR Path="/6019DBCE/60198F29" Ref="#PWR037"  Part="1"
 AR Path="/601B4C19/60198F29" Ref="#PWR067"  Part="1"
-F 0 "#PWR067" H 5450 3950 50  0001 C CNN
+F 0 "#PWR037" H 5450 3950 50  0001 C CNN
 F 1 "GND" H 5455 4027 50  0000 C CNN
 F 2 "" H 5450 4200 50  0001 C CNN
@@
 AR Path="/6019DBCE/6019E3AD" Ref="R28"  Part="1"
 AR Path="/601B4C19/6019E3AD" Ref="R64"  Part="1"
-F 0 "R64" H 1520 1996 50  0000 L CNN
+F 0 "R28" H 1520 1996 50  0000 L CNN
 F 1 "330" H 1520 1905 50  0000 L CNN
 F 2 "Resistor_THT:R_Axial_DIN0204_L3.6mm_D1.6mm_P5.08mm_Horizontal" V 1380 1950 50  0001 C CNN
@@
 AR Path="/6019DBCE/6019E3AF" Ref="#PWR033"  Part="1"
 AR Path="/601B4C19/6019E3AF" Ref="#PWR063"  Part="1"
-F 0 "#PWR063" H 1450 2800 50  0001 C CNN
+F 0 "#PWR033" H 1450 2800 50  0001 C CNN
 F 1 "GND" H 1455 2877 50  0000 C CNN
 F 2 "" H 1450 3050 50  0001 C CNN
@@
 AR Path="/6019DBCE/6019E3AA" Ref="R29"  Part="1"
 AR Path="/601B4C19/6019E3AA" Ref="R65"  Part="1"
-F 0 "R65" H 1520 2946 50  0000 L CNN
+F 0 "R29" H 1520 2946 50  0000 L CNN
 F 1 "330" H 1520 2855 50  0000 L CNN
 F 2 "Resistor_THT:R_Axial_DIN0204_L3.6mm_D1.6mm_P5.08mm_Horizontal" V 1380 2900 50  0001 C CNN
@@
 AR Path="/6019DBCE/6019E3B1" Ref="#PWR034"  Part="1"
 AR Path="/601B4C19/6019E3B1" Ref="#PWR064"  Part="1"
-F 0 "#PWR064" H 1450 3800 50  0001 C CNN
+F 0 "#PWR034" H 1450 3800 50  0001 C CNN
 F 1 "GND" H 1455 3877 50  0000 C CNN
 F 2 "" H 1450 4050 50  0001 C CNN
@@
 AR Path="/6019DBCE/60198F3A" Ref="R30"  Part="1"
 AR Path="/601B4C19/60198F3A" Ref="R66"  Part="1"
-F 0 "R66" H 1520 3946 50  0000 L CNN
+F 0 "R30" H 1520 3946 50  0000 L CNN
 F 1 "330" H 1520 3855 50  0000 L CNN
 F 2 "Resistor_THT:R_Axial_DIN0204_L3.6mm_D1.6mm_P5.08mm_Horizontal" V 1380 3900 50  0001 C CNN
@@
 AR Path="/6019DBCE/6019A6B5" Ref="U14"  Part="2"
 AR Path="/601B4C19/6019A6B5" Ref="U24"  Part="2"
-F 0 "U24" H 1508 3884 50  0000 L CNN
+F 0 "U14" H 1508 3884 50  0000 L CNN
 F 1 "screw_term" H 1508 3793 50  0000 L CNN
 F 2 "Connector_PinHeader_1.27mm:PinHeader_1x02_P1.27mm_Vertical" H 1450 3750 50  0001 C CNN
@@
 AR Path="/6019DBCE/6019E3B7" Ref="U13"  Part="2"
 AR Path="/601B4C19/6019E3B7" Ref="U23"  Part="2"
-F 0 "U23" H 1508 1934 50  0000 L CNN
+F 0 "U13" H 1508 1934 50  0000 L CNN
 F 1 "screw_term" H 1508 1843 50  0000 L CNN
 F 2 "Connector_PinHeader_1.27mm:PinHeader_1x02_P1.27mm_Vertical" H 1450 1800 50  0001 C CNN
@@
 AR Path="/6019DBCE/6019E3B0" Ref="U13"  Part="1"
 AR Path="/601B4C19/6019E3B0" Ref="U23"  Part="1"
-F 0 "U23" H 1508 2884 50  0000 L CNN
+F 0 "U13" H 1508 2884 50  0000 L CNN
 F 1 "screw_term" H 1508 2793 50  0000 L CNN
 F 2 "Connector_PinHeader_1.27mm:PinHeader_1x02_P1.27mm_Vertical" H 1450 2750 50  0001 C CNN
@@
 AR Path="/6019DBCE/6019E3AE" Ref="#U010"  Part="2"
 AR Path="/601B4C19/6019E3AE" Ref="#U021"  Part="2"
-F 0 "#U021" H 3375 2515 50  0000 C CNN
+F 0 "#U010" H 3375 2515 50  0000 C CNN
 F 1 "Mux" H 3375 2424 50  0000 C CNN
 F 2 "" H 3350 2050 50  0001 C CNN
@@
 AR Path="/6019DBCE/6017E42E" Ref="U12"  Part="4"
 AR Path="/601B4C19/6017E42E" Ref="U7"  Part="4"
-F 0 "U7" H 6000 3433 50  0000 C CNN
+F 0 "U12" H 6000 3433 50  0000 C CNN
 F 1 "TL084" H 6000 3524 50  0000 C CNN
-F 2 "" H 5950 3900 50  0001 C CNN
+F 2 "Package_DIP:DIP-14_W7.62mm" H 5950 3900 50  0001 C CNN
 F 3 "http://www.ti.com/lit/ds/symlink/tl081.pdf" H 6050 4000 50  0001 C CNN
 	4    6000 3800

Commit message: updated all mux packages in eeschema
Changed lines of the file:
@@
 $Descr A4 11693 8268
 encoding utf-8
-Sheet 5 11
+Sheet 9 11
 Title ""
 Date ""
@@
 AR Path="/6019DBCE/60198F27" Ref="#PWR032"  Part="1"
 AR Path="/601B4C19/60198F27" Ref="#PWR062"  Part="1"
-F 0 "#PWR032" H 1450 1850 50  0001 C CNN
+F 0 "#PWR062" H 1450 1850 50  0001 C CNN
 F 1 "GND" H 1455 1927 50  0000 C CNN
 F 2 "" H 1450 2100 50  0001 C CNN
@@
 AR Path="/6019DBCE/6015EF5C" Ref="R35"  Part="1"
 AR Path="/601B4C19/6015EF5C" Ref="R71"  Part="1"
-F 0 "R35" H 5520 4096 50  0000 L CNN
+F 0 "R71" H 5520 4096 50  0000 L CNN
 F 1 "15" H 5520 4005 50  0000 L CNN
 F 2 "Resistor_THT:R_Axial_DIN0204_L3.6mm_D1.6mm_P5.08mm_Horizontal" V 5380 4050 50  0001 C CNN
@@
 AR Path="/6019DBCE/6019E3A7" Ref="R36"  Part="1"
 AR Path="/601B4C19/6019E3A7" Ref="R72"  Part="1"
-F 0 "R36" V 5743 3250 50  0000 C CNN
+F 0 "R72" V 5743 3250 50  0000 C CNN
 F 1 "15" V 5834 3250 50  0000 C CNN
 F 2 "Resistor_THT:R_Axial_DIN0204_L3.6mm_D1.6mm_P5.08mm_Horizontal" V 5880 3250 50  0001 C CNN
@@
 AR Path="/6019DBCE/6019E3B2" Ref="R33"  Part="1"
 AR Path="/601B4C19/6019E3B2" Ref="R69"  Part="1"
-F 0 "R33" V 5307 3700 50  0000 C CNN
+F 0 "R69" V 5307 3700 50  0000 C CNN
 F 1 "1" V 5216 3700 50  0000 C CNN
 F 2 "Resistor_THT:R_Axial_DIN0204_L3.6mm_D1.6mm_P5.08mm_Horizontal" V 5030 3700 50  0001 C CNN
@@
 AR Path="/6019DBCE/6019E3A8" Ref="R34"  Part="1"
 AR Path="/601B4C19/6019E3A8" Ref="R70"  Part="1"
-F 0 "R34" V 5000 3900 50  0000 C CNN
+F 0 "R70" V 5000 3900 50  0000 C CNN
 F 1 "1" V 4900 3900 50  0000 C CNN
 F 2 "Resistor_THT:R_Axial_DIN0204_L3.6mm_D1.6mm_P5.08mm_Horizontal" V 5030 3900 50  0001 C CNN
@@
 AR Path="/6019DBCE/6019E3B3" Ref="R31"  Part="1"
 AR Path="/601B4C19/6019E3B3" Ref="R67"  Part="1"
-F 0 "R31" H 3320 3546 50  0000 L CNN
+F 0 "R67" H 3320 3546 50  0000 L CNN
 F 1 "330" H 3320 3455 50  0000 L CNN
 F 2 "Resistor_THT:R_Axial_DIN0204_L3.6mm_D1.6mm_P5.08mm_Horizontal" V 3180 3500 50  0001 C CNN
@@
 AR Path="/6019DBCE/60198F36" Ref="R32"  Part="1"
 AR Path="/601B4C19/60198F36" Ref="R68"  Part="1"
-F 0 "R32" H 3320 3846 50  0000 L CNN
+F 0 "R68" H 3320 3846 50  0000 L CNN
 F 1 "560" H 3320 3755 50  0000 L CNN
 F 2 "Resistor_THT:R_Axial_DIN0204_L3.6mm_D1.6mm_P5.08mm_Horizontal" V 3180 3800 50  0001 C CNN
@@
 AR Path="/6019DBCE/60198F37" Ref="#PWR035"  Part="1"
 AR Path="/601B4C19/60198F37" Ref="#PWR065"  Part="1"
-F 0 "#PWR035" H 3250 3200 50  0001 C CNN
+F 0 "#PWR065" H 3250 3200 50  0001 C CNN
 F 1 "+3.3V" H 3265 3523 50  0000 C CNN
 F 2 "" H 3250 3350 50  0001 C CNN
@@
 AR Path="/6019DBCE/6019E3A9" Ref="#PWR036"  Part="1"
 AR Path="/601B4C19/6019E3A9" Ref="#PWR066"  Part="1"
-F 0 "#PWR036" H 3250 3700 50  0001 C CNN
+F 0 "#PWR066" H 3250 3700 50  0001 C CNN
 F 1 "GND" H 3255 3777 50  0000 C CNN
 F 2 "" H 3250 3950 50  0001 C CNN
@@
 AR Path="/6019DBCE/60198F29" Ref="#PWR037"  Part="1"
 AR Path="/601B4C19/60198F29" Ref="#PWR067"  Part="1"
-F 0 "#PWR037" H 5450 3950 50  0001 C CNN
+F 0 "#PWR067" H 5450 3950 50  0001 C CNN
 F 1 "GND" H 5455 4027 50  0000 C CNN
 F 2 "" H 5450 4200 50  0001 C CNN
@@
 AR Path="/6019DBCE/6019E3AD" Ref="R28"  Part="1"
 AR Path="/601B4C19/6019E3AD" Ref="R64"  Part="1"
-F 0 "R28" H 1520 1996 50  0000 L CNN
+F 0 "R64" H 1520 1996 50  0000 L CNN
 F 1 "330" H 1520 1905 50  0000 L CNN
 F 2 "Resistor_THT:R_Axial_DIN0204_L3.6mm_D1.6mm_P5.08mm_Horizontal" V 1380 1950 50  0001 C CNN
@@
 AR Path="/6019DBCE/6019E3AF" Ref="#PWR033"  Part="1"
 AR Path="/601B4C19/6019E3AF" Ref="#PWR063"  Part="1"
-F 0 "#PWR033" H 1450 2800 50  0001 C CNN
+F 0 "#PWR063" H 1450 2800 50  0001 C CNN
 F 1 "GND" H 1455 2877 50  0000 C CNN
 F 2 "" H 1450 3050 50  0001 C CNN
@@
 AR Path="/6019DBCE/6019E3AA" Ref="R29"  Part="1"
 AR Path="/601B4C19/6019E3AA" Ref="R65"  Part="1"
-F 0 "R29" H 1520 2946 50  0000 L CNN
+F 0 "R65" H 1520 2946 50  0000 L CNN
 F 1 "330" H 1520 2855 50  0000 L CNN
 F 2 "Resistor_THT:R_Axial_DIN0204_L3.6mm_D1.6mm_P5.08mm_Horizontal" V 1380 2900 50  0001 C CNN
@@
 AR Path="/6019DBCE/6019E3B1" Ref="#PWR034"  Part="1"
 AR Path="/601B4C19/6019E3B1" Ref="#PWR064"  Part="1"
-F 0 "#PWR034" H 1450 3800 50  0001 C CNN
+F 0 "#PWR064" H 1450 3800 50  0001 C CNN
 F 1 "GND" H 1455 3877 50  0000 C CNN
 F 2 "" H 1450 4050 50  0001 C CNN
@@
 AR Path="/6019DBCE/60198F3A" Ref="R30"  Part="1"
 AR Path="/601B4C19/60198F3A" Ref="R66"  Part="1"
-F 0 "R30" H 1520 3946 50  0000 L CNN
+F 0 "R66" H 1520 3946 50  0000 L CNN
 F 1 "330" H 1520 3855 50  0000 L CNN
 F 2 "Resistor_THT:R_Axial_DIN0204_L3.6mm_D1.6mm_P5.08mm_Horizontal" V 1380 3900 50  0001 C CNN
@@
 AR Path="/6019DBCE/6019A6B5" Ref="U14"  Part="2"
 AR Path="/601B4C19/6019A6B5" Ref="U24"  Part="2"
-F 0 "U14" H 1508 3884 50  0000 L CNN
+F 0 "U24" H 1508 3884 50  0000 L CNN
 F 1 "screw_term" H 1508 3793 50  0000 L CNN
 F 2 "Connector_PinHeader_1.27mm:PinHeader_1x02_P1.27mm_Vertical" H 1450 3750 50  0001 C CNN
@@
 AR Path="/6019DBCE/6019E3B7" Ref="U13"  Part="2"
 AR Path="/601B4C19/6019E3B7" Ref="U23"  Part="2"
-F 0 "U13" H 1508 1934 50  0000 L CNN
+F 0 "U23" H 1508 1934 50  0000 L CNN
 F 1 "screw_term" H 1508 1843 50  0000 L CNN
 F 2 "Connector_PinHeader_1.27mm:PinHeader_1x02_P1.27mm_Vertical" H 1450 1800 50  0001 C CNN
@@
 AR Path="/6019DBCE/6019E3B0" Ref="U13"  Part="1"
 AR Path="/601B4C19/6019E3B0" Ref="U23"  Part="1"
-F 0 "U13" H 1508 2884 50  0000 L CNN
+F 0 "U23" H 1508 2884 50  0000 L CNN
 F 1 "screw_term" H 1508 2793 50  0000 L CNN
 F 2 "Connector_PinHeader_1.27mm:PinHeader_1x02_P1.27mm_Vertical" H 1450 2750 50  0001 C CNN
@@
 AR Path="/6019DBCE/6019E3AE" Ref="#U010"  Part="2"
 AR Path="/601B4C19/6019E3AE" Ref="#U021"  Part="2"
-F 0 "#U010" H 3375 2515 50  0000 C CNN
+F 0 "#U021" H 3375 2515 50  0000 C CNN
 F 1 "Mux" H 3375 2424 50  0000 C CNN
-F 2 "" H 3350 2050 50  0001 C CNN
+F 2 "Package_DIP:DIP-16_W7.62mm" H 3350 2050 50  0001 C CNN
 F 3 "http://www.ti.com/lit/ds/symlink/tl081.pdf" H 3350 2050 50  0001 C CNN
 	2    3350 2050
@@
 AR Path="/6019DBCE/6017E42E" Ref="U12"  Part="4"
 AR Path="/601B4C19/6017E42E" Ref="U7"  Part="4"
-F 0 "U12" H 6000 3433 50  0000 C CNN
+F 0 "U7" H 6000 3433 50  0000 C CNN
 F 1 "TL084" H 6000 3524 50  0000 C CNN
 F 2 "Package_DIP:DIP-14_W7.62mm" H 5950 3900 50  0001 C CNN

Commit message: added all muxes to the board
Parts:
- added U10: Mux, Package_DIP:DIP-16_W7.62mm, symbol PNG_PCB_Parts:Mux
- renumbered U14 to U11, U13 to U11, U12 to U6, U13 to U9
Connections:
- net V1: now also U10.3 (yout)
- net mux0: now also U10.1 (y0)
- net mux1: now also U10.5 (y1)
- net mux2: now also U10.2 (y2)
Changed lines of the file:
@@
 AR Path="/6017DA21/6019A6B5" Ref="U?"  Part="1"
 AR Path="/601927EB/6019A6B5" Ref="U?"  Part="2"
-AR Path="/6019DBCE/6019A6B5" Ref="U14"  Part="2"
-AR Path="/601B4C19/6019A6B5" Ref="U24"  Part="2"
-F 0 "U24" H 1508 3884 50  0000 L CNN
+AR Path="/6019DBCE/6019A6B5" Ref="U11"  Part="2"
+AR Path="/601B4C19/6019A6B5" Ref="U20"  Part="2"
+F 0 "U20" H 1508 3884 50  0000 L CNN
 F 1 "screw_term" H 1508 3793 50  0000 L CNN
 F 2 "Connector_PinHeader_1.27mm:PinHeader_1x02_P1.27mm_Vertical" H 1450 3750 50  0001 C CNN
@@
 AR Path="/601927EB/6019A2A3" Ref="U?"  Part="2"
 AR Path="/6019DBCE/6019A2A3" Ref="U?"  Part="2"
-AR Path="/6019DBCE/6019E3B7" Ref="U13"  Part="2"
-AR Path="/601B4C19/6019E3B7" Ref="U23"  Part="2"
-F 0 "U23" H 1508 1934 50  0000 L CNN
+AR Path="/6019DBCE/6019E3B7" Ref="U9"  Part="2"
+AR Path="/601B4C19/6019E3B7" Ref="U18"  Part="2"
+F 0 "U18" H 1508 1934 50  0000 L CNN
 F 1 "screw_term" H 1508 1843 50  0000 L CNN
 F 2 "Connector_PinHeader_1.27mm:PinHeader_1x02_P1.27mm_Vertical" H 1450 1800 50  0001 C CNN
@@
 AR Path="/601927EB/60198F2E" Ref="U?"  Part="1"
 AR Path="/6019DBCE/60198F2E" Ref="U?"  Part="1"
-AR Path="/6019DBCE/6019E3B0" Ref="U13"  Part="1"
-AR Path="/601B4C19/6019E3B0" Ref="U23"  Part="1"
-F 0 "U23" H 1508 2884 50  0000 L CNN
+AR Path="/6019DBCE/6019E3B0" Ref="U11"  Part="1"
+AR Path="/601B4C19/6019E3B0" Ref="U20"  Part="1"
+F 0 "U20" H 1508 2884 50  0000 L CNN
 F 1 "screw_term" H 1508 2793 50  0000 L CNN
 F 2 "Connector_PinHeader_1.27mm:PinHeader_1x02_P1.27mm_Vertical" H 1450 2750 50  0001 C CNN
 F 3 "" H 1450 2750 50  0001 C CNN
 	1    1450 2750
-	1    0    0    -1
-$EndComp
-$Comp
-L PNG_PCB_Parts:Mux U?
-U 2 1 6019E3AE
-P 3350 2050
-AR Path="/60132BC3/6013AE22/60198F2C" Ref="U?"  Part="1"
-AR Path="/6017CC5E/60198F2C" Ref="U?"  Part="1"
-AR Path="/6017DA21/60198F2C" Ref="U?"  Part="1"
-AR Path="/601927EB/60198F2C" Ref="U?"  Part="2"
-AR Path="/6019DBCE/60198F2C" Ref="U?"  Part="2"
-AR Path="/6019DBCE/6019E3AE" Ref="#U010"  Part="2"
-AR Path="/601B4C19/6019E3AE" Ref="#U021"  Part="2"
-F 0 "#U021" H 3375 2515 50  0000 C CNN
-F 1 "Mux" H 3375 2424 50  0000 C CNN
-F 2 "Package_DIP:DIP-16_W7.62mm" H 3350 2050 50  0001 C CNN
-F 3 "http://www.ti.com/lit/ds/symlink/tl081.pdf" H 3350 2050 50  0001 C CNN
-	2    3350 2050
 	1    0    0    -1
 $EndComp
@@
 AR Path="/6017DA21/6017E42E" Ref="U?"  Part="1"
 AR Path="/601927EB/6017E42E" Ref="U?"  Part="2"
-AR Path="/6019DBCE/6017E42E" Ref="U12"  Part="4"
-AR Path="/601B4C19/6017E42E" Ref="U7"  Part="4"
-F 0 "U7" H 6000 3433 50  0000 C CNN
+AR Path="/6019DBCE/6017E42E" Ref="U6"  Part="4"
+AR Path="/601B4C19/6017E42E" Ref="U15"  Part="4"
+F 0 "U15" H 6000 3433 50  0000 C CNN
 F 1 "TL084" H 6000 3524 50  0000 C CNN
 F 2 "Package_DIP:DIP-14_W7.62mm" H 5950 3900 50  0001 C CNN
@@
 	1    0    0    1
 $EndComp
+$Comp
+L PNG_PCB_Parts:Mux U10
+U 2 1 6017A5CD
+P 3350 2050
+AR Path="/6019DBCE/6017A5CD" Ref="U10"  Part="2"
+AR Path="/601B4C19/6017A5CD" Ref="U19"  Part="2"
+F 0 "U19" H 3375 2515 50  0000 C CNN
+F 1 "Mux" H 3375 2424 50  0000 C CNN
+F 2 "Package_DIP:DIP-16_W7.62mm" H 3350 2050 50  0001 C CNN
+F 3 "" H 3350 2050 50  0001 C CNN
+	2    3350 2050
+	1    0    0    -1
+$EndComp
 $EndSCHEMATC
