File: ampA.sch (KiCad schematic (older format))
At the start: 8 parts, among them U3 Mux, U4 MCP6004

Commit message: revised sensor connector
Parts:
- R1: value 330 -> 560
- R2: value 560 -> 300
- renumbered U3 to U2, U4 to U3
Changed lines of the file:
@@
 $Descr A4 11693 8268
 encoding utf-8
-Sheet 2 41
+Sheet 18 41
 Title ""
 Date ""
@@
 AR Path="/601927EB/6019D565" Ref="R?"  Part="1"
 AR Path="/6019C043/6019D565" Ref="R?"  Part="1"
-AR Path="/601B4C0E/6019D565" Ref="R65"  Part="1"
-AR Path="/601B73B7/6019D565" Ref="R125"  Part="1"
-F 0 "R5" H 5520 4096 50  0000 L CNN
+AR Path="/601B4C0E/6019D565" Ref="R41"  Part="1"
+AR Path="/601B73B7/6019D565" Ref="R77"  Part="1"
+F 0 "R77" H 5520 4096 50  0000 L CNN
 F 1 "15" H 5520 4005 50  0000 L CNN
 F 2 "Resistor_THT:R_Axial_DIN0204_L3.6mm_D1.6mm_P5.08mm_Horizontal" V 5380 4050 50  0001 C CNN
@@
 AR Path="/601927EB/60198F32" Ref="R?"  Part="1"
 AR Path="/6019C043/60198F32" Ref="R?"  Part="1"
-AR Path="/601B4C0E/60198F32" Ref="R66"  Part="1"
-AR Path="/601B73B7/60198F32" Ref="R126"  Part="1"
-F 0 "R6" V 5743 3250 50  0000 C CNN
+AR Path="/601B4C0E/60198F32" Ref="R42"  Part="1"
+AR Path="/601B73B7/60198F32" Ref="R78"  Part="1"
+F 0 "R78" V 5743 3250 50  0000 C CNN
 F 1 "15" V 5834 3250 50  0000 C CNN
 F 2 "Resistor_THT:R_Axial_DIN0204_L3.6mm_D1.6mm_P5.08mm_Horizontal" V 5880 3250 50  0001 C CNN
@@
 AR Path="/601927EB/6017E431" Ref="R?"  Part="1"
 AR Path="/6019C043/6017E431" Ref="R?"  Part="1"
-AR Path="/601B4C0E/6017E431" Ref="R63"  Part="1"
-AR Path="/601B73B7/6017E431" Ref="R123"  Part="1"
-F 0 "R3" V 5307 3700 50  0000 C CNN
+AR Path="/601B4C0E/6017E431" Ref="R39"  Part="1"
+AR Path="/601B73B7/6017E431" Ref="R75"  Part="1"
+F 0 "R75" V 5307 3700 50  0000 C CNN
 F 1 "1" V 5216 3700 50  0000 C CNN
 F 2 "Resistor_THT:R_Axial_DIN0204_L3.6mm_D1.6mm_P5.08mm_Horizontal" V 5030 3700 50  0001 C CNN
@@
 AR Path="/601927EB/6019D568" Ref="R?"  Part="1"
 AR Path="/6019C043/6019D568" Ref="R?"  Part="1"
-AR Path="/601B4C0E/6019D568" Ref="R64"  Part="1"
-AR Path="/601B73B7/6019D568" Ref="R124"  Part="1"
-F 0 "R4" V 5000 3900 50  0000 C CNN
+AR Path="/601B4C0E/6019D568" Ref="R40"  Part="1"
+AR Path="/601B73B7/6019D568" Ref="R76"  Part="1"
+F 0 "R76" V 5000 3900 50  0000 C CNN
 F 1 "1" V 4900 3900 50  0000 C CNN
 F 2 "Resistor_THT:R_Axial_DIN0204_L3.6mm_D1.6mm_P5.08mm_Horizontal" V 5030 3900 50  0001 C CNN
@@
 AR Path="/601927EB/6019D55E" Ref="R?"  Part="1"
 AR Path="/6019C043/6019D55E" Ref="R?"  Part="1"
-AR Path="/601B4C0E/6019D55E" Ref="R61"  Part="1"
-AR Path="/601B73B7/6019D55E" Ref="R121"  Part="1"
-F 0 "R1" H 3320 3546 50  0000 L CNN
-F 1 "330" H 3320 3455 50  0000 L CNN
+AR Path="/601B4C0E/6019D55E" Ref="R37"  Part="1"
+AR Path="/601B73B7/6019D55E" Ref="R73"  Part="1"
+F 0 "R73" H 3320 3546 50  0000 L CNN
+F 1 "560" H 3320 3455 50  0000 L CNN
 F 2 "Resistor_THT:R_Axial_DIN0204_L3.6mm_D1.6mm_P5.08mm_Horizontal" V 3180 3500 50  0001 C CNN
 F 3 "~" H 3250 3500 50  0001 C CNN
@@
 AR Path="/601927EB/6019D55F" Ref="R?"  Part="1"
 AR Path="/6019C043/6019D55F" Ref="R?"  Part="1"
-AR Path="/601B4C0E/6019D55F" Ref="R62"  Part="1"
-AR Path="/601B73B7/6019D55F" Ref="R122"  Part="1"
-F 0 "R2" H 3320 3846 50  0000 L CNN
-F 1 "560" H 3320 3755 50  0000 L CNN
+AR Path="/601B4C0E/6019D55F" Ref="R38"  Part="1"
+AR Path="/601B73B7/6019D55F" Ref="R74"  Part="1"
+F 0 "R74" H 3320 3846 50  0000 L CNN
+F 1 "300" H 3320 3755 50  0000 L CNN
 F 2 "Resistor_THT:R_Axial_DIN0204_L3.6mm_D1.6mm_P5.08mm_Horizontal" V 3180 3800 50  0001 C CNN
 F 3 "~" H 3250 3800 50  0001 C CNN
 	1    3250 3800
-	1    0    0    -1
-$EndComp
-$Comp
-L power:+3.3V #PWR?
-U 1 1 6019D560
-P 3250 3350
-AR Path="/60132BC3/6013AE22/6019D560" Ref="#PWR?"  Part="1"
-AR Path="/6017CC5E/6019D560" Ref="#PWR08"  Part="1"
-AR Path="/6017DA21/6019D560" Ref="#PWR?"  Part="1"
-AR Path="/601927EB/6019D560" Ref="#PWR?"  Part="1"
-AR Path="/6019C043/6019D560" Ref="#PWR?"  Part="1"
-AR Path="/601B4C0E/6019D560" Ref="#PWR098"  Part="1"
-AR Path="/601B73B7/6019D560" Ref="#PWR0188"  Part="1"
-F 0 "#PWR0188" H 3250 3200 50  0001 C CNN
-F 1 "+3.3V" H 3265 3523 50  0000 C CNN
-F 2 "" H 3250 3350 50  0001 C CNN
-F 3 "" H 3250 3350 50  0001 C CNN
-	1    3250 3350
 	1    0    0    -1
 $EndComp
@@
 AR Path="/601927EB/60198F38" Ref="#PWR?"  Part="1"
 AR Path="/6019C043/60198F38" Ref="#PWR?"  Part="1"
-AR Path="/601B4C0E/60198F38" Ref="#PWR099"  Part="1"
-AR Path="/601B73B7/60198F38" Ref="#PWR0189"  Part="1"
-F 0 "#PWR0189" H 3250 3700 50  0001 C CNN
+AR Path="/601B4C0E/60198F38" Ref="#PWR051"  Part="1"
+AR Path="/601B73B7/60198F38" Ref="#PWR093"  Part="1"
+F 0 "#PWR093" H 3250 3700 50  0001 C CNN
 F 1 "GND" H 3255 3777 50  0000 C CNN
 F 2 "" H 3250 3950 50  0001 C CNN
@@
 AR Path="/601927EB/6016B854" Ref="#PWR?"  Part="1"
 AR Path="/6019C043/6016B854" Ref="#PWR?"  Part="1"
-AR Path="/601B4C0E/6016B854" Ref="#PWR0100"  Part="1"
-AR Path="/601B73B7/6016B854" Ref="#PWR0190"  Part="1"
-F 0 "#PWR0190" H 5450 3950 50  0001 C CNN
+AR Path="/601B4C0E/6016B854" Ref="#PWR052"  Part="1"
+AR Path="/601B73B7/6016B854" Ref="#PWR094"  Part="1"
+F 0 "#PWR094" H 5450 3950 50  0001 C CNN
 F 1 "GND" H 5455 4027 50  0000 C CNN
 F 2 "" H 5450 4200 50  0001 C CNN
@@
 AR Path="/601927EB/601899DD" Ref="#PWR?"  Part="1"
 AR Path="/6019C043/601899DD" Ref="#PWR?"  Part="1"
-AR Path="/601B4C0E/601899DD" Ref="#PWR0102"  Part="1"
-AR Path="/601B73B7/601899DD" Ref="#PWR0192"  Part="1"
-F 0 "#PWR0192" H 5700 2050 50  0001 C CNN
+AR Path="/601B4C0E/601899DD" Ref="#PWR054"  Part="1"
+AR Path="/601B73B7/601899DD" Ref="#PWR096"  Part="1"
+F 0 "#PWR096" H 5700 2050 50  0001 C CNN
 F 1 "GND" H 5705 2127 50  0000 C CNN
 F 2 "" H 5700 2300 50  0001 C CNN
@@
 AR Path="/601927EB/60189E9E" Ref="#PWR?"  Part="1"
 AR Path="/6019C043/60189E9E" Ref="#PWR?"  Part="1"
-AR Path="/601B4C0E/60189E9E" Ref="#PWR0101"  Part="1"
-AR Path="/601B73B7/60189E9E" Ref="#PWR0191"  Part="1"
-F 0 "#PWR0191" H 5700 1600 50  0001 C CNN
+AR Path="/601B4C0E/60189E9E" Ref="#PWR053"  Part="1"
+AR Path="/601B73B7/60189E9E" Ref="#PWR095"  Part="1"
+F 0 "#PWR095" H 5700 1600 50  0001 C CNN
 F 1 "+3.3V" H 5715 1923 50  0000 C CNN
 F 2 "" H 5700 1750 50  0001 C CNN
@@
 AR Path="/601927EB/60195FF1" Ref="#PWR?"  Part="1"
 AR Path="/6019C043/60195FF1" Ref="#PWR?"  Part="1"
-AR Path="/601B4C0E/60195FF1" Ref="#PWR0104"  Part="1"
-AR Path="/601B73B7/60195FF1" Ref="#PWR0194"  Part="1"
-F 0 "#PWR0194" H 7150 2100 50  0001 C CNN
+AR Path="/601B4C0E/60195FF1" Ref="#PWR056"  Part="1"
+AR Path="/601B73B7/60195FF1" Ref="#PWR098"  Part="1"
+F 0 "#PWR098" H 7150 2100 50  0001 C CNN
 F 1 "GND" H 7155 2177 50  0000 C CNN
 F 2 "" H 7150 2350 50  0001 C CNN
@@
 AR Path="/601927EB/60198969" Ref="#PWR?"  Part="1"
 AR Path="/6019C043/60198969" Ref="#PWR?"  Part="1"
-AR Path="/601B4C0E/60198969" Ref="#PWR0103"  Part="1"
-AR Path="/601B73B7/60198969" Ref="#PWR0193"  Part="1"
-F 0 "#PWR0193" H 7150 1600 50  0001 C CNN
+AR Path="/601B4C0E/60198969" Ref="#PWR055"  Part="1"
+AR Path="/601B73B7/60198969" Ref="#PWR097"  Part="1"
+F 0 "#PWR097" H 7150 1600 50  0001 C CNN
 F 1 "+3.3V" H 7165 1923 50  0000 C CNN
 F 2 "" H 7150 1750 50  0001 C CNN
@@
 $EndComp
 $Comp
-L PNG_PCB_Parts:Mux U3
+L PNG_PCB_Parts:Mux U2
 U 1 1 6016DEDC
 P 3350 2050
-AR Path="/6017CC5E/6016DEDC" Ref="U3"  Part="1"
-AR Path="/601B4C0E/6016DEDC" Ref="U6"  Part="1"
-AR Path="/601B73B7/6016DEDC" Ref="U9"  Part="1"
-F 0 "U3" H 3375 2515 50  0000 C CNN
+AR Path="/6017CC5E/6016DEDC" Ref="U2"  Part="1"
+AR Path="/601B4C0E/6016DEDC" Ref="U5"  Part="1"
+AR Path="/601B73B7/6016DEDC" Ref="U8"  Part="1"
+F 0 "U8" H 3375 2515 50  0000 C CNN
 F 1 "Mux" H 3375 2424 50  0000 C CNN
 F 2 "Package_DIP:DIP-16_W7.62mm" H 3350 2050 50  0001 C CNN
@@
 $EndComp
 $Comp
-L PNG_PCB_Parts:Mux U3
+L PNG_PCB_Parts:Mux U2
 U 3 1 6016F806
 P 5700 2100
-AR Path="/6017CC5E/6016F806" Ref="U3"  Part="3"
-AR Path="/601B4C0E/6016F806" Ref="U6"  Part="3"
-AR Path="/601B73B7/6016F806" Ref="U9"  Part="3"
-F 0 "U3" H 5928 2221 50  0000 L CNN
+AR Path="/6017CC5E/6016F806" Ref="U2"  Part="3"
+AR Path="/601B4C0E/6016F806" Ref="U5"  Part="3"
+AR Path="/601B73B7/6016F806" Ref="U8"  Part="3"
+F 0 "U8" H 5928 2221 50  0000 L CNN
 F 1 "Mux" H 5928 2130 50  0000 L CNN
 F 2 "Package_DIP:DIP-16_W7.62mm" H 5700 2100 50  0001 C CNN
@@
 $EndComp
 $Comp
-L Amplifier_Operational:MCP6004 U4
+L Amplifier_Operational:MCP6004 U3
 U 1 1 60189002
 P 6000 3800
-AR Path="/6017CC5E/60189002" Ref="U4"  Part="1"
-AR Path="/601B4C0E/60189002" Ref="U7"  Part="1"
-AR Path="/601B73B7/60189002" Ref="U10"  Part="1"
-F 0 "U4" H 6000 4167 50  0000 C CNN
+AR Path="/6017CC5E/60189002" Ref="U3"  Part="1"
+AR Path="/601B4C0E/60189002" Ref="U6"  Part="1"
+AR Path="/601B73B7/60189002" Ref="U9"  Part="1"
+F 0 "U9" H 6000 4167 50  0000 C CNN
 F 1 "MCP6004" H 6000 4076 50  0000 C CNN
 F 2 "Package_DIP:DIP-14_W7.62mm" H 5950 3900 50  0001 C CNN
@@
 $EndComp
 $Comp
-L Amplifier_Operational:MCP6004 U4
+L Amplifier_Operational:MCP6004 U3
 U 5 1 6018B5B8
 P 7250 2050
-AR Path="/6017CC5E/6018B5B8" Ref="U4"  Part="5"
-AR Path="/601B4C0E/6018B5B8" Ref="U7"  Part="5"
-AR Path="/601B73B7/6018B5B8" Ref="U10"  Part="5"
-F 0 "U4" H 7208 2096 50  0000 L CNN
+AR Path="/6017CC5E/6018B5B8" Ref="U3"  Part="5"
+AR Path="/601B4C0E/6018B5B8" Ref="U6"  Part="5"
+AR Path="/601B73B7/6018B5B8" Ref="U9"  Part="5"
+F 0 "U9" H 7208 2096 50  0000 L CNN
 F 1 "MCP6004" H 7208 2005 50  0000 L CNN
 F 2 "Package_DIP:DIP-14_W7.62mm" H 7200 2150 50  0001 C CNN
@@
 F2 "Vsense" I R 1550 3200 50
 $EndSheet
+$Comp
+L power:+3.3V #PWR?
+U 1 1 6019D560
+P 3250 3350
+AR Path="/60132BC3/6013AE22/6019D560" Ref="#PWR?"  Part="1"
+AR Path="/6017CC5E/6019D560" Ref="#PWR08"  Part="1"
+AR Path="/6017DA21/6019D560" Ref="#PWR?"  Part="1"
+AR Path="/601927EB/6019D560" Ref="#PWR?"  Part="1"
+AR Path="/6019C043/6019D560" Ref="#PWR?"  Part="1"
+AR Path="/601B4C0E/6019D560" Ref="#PWR050"  Part="1"
+AR Path="/601B73B7/6019D560" Ref="#PWR092"  Part="1"
+F 0 "#PWR092" H 3250 3200 50  0001 C CNN
+F 1 "+3.3V" H 3265 3523 50  0000 C CNN
+F 2 "" H 3250 3350 50  0001 C CNN
+F 3 "" H 3250 3350 50  0001 C CNN
+	1    3250 3350
+	1    0    0    -1
+$EndComp
 $EndSCHEMATC

Commit message: moved sensor r div to other side of mux
Parts:
- added R3: 560, Resistor_THT:R_Axial_DIN0204_L3.6mm_D1.6mm_P5.08mm_Horizontal, symbol Device:R
- renumbered R3 to R4, R4 to R5, R5 to R6, R6 to R7
Connections:
- net +3V3: now also R3.1
- net V1: now also R3.2

Commit message: updated mcp6004 footprint on sch
Parts:
- U3: footprint Package_DIP:DIP-14_W7.62mm -> Package_SO:SOIC-16_4.55x10.3mm_P1.27mm
Changed lines of the file:
@@
 F 0 "U3" H 6000 4167 50  0000 C CNN
 F 1 "MCP6004" H 6000 4076 50  0000 C CNN
-F 2 "Package_DIP:DIP-14_W7.62mm" H 5950 3900 50  0001 C CNN
+F 2 "Package_SO:SOIC-16_4.55x10.3mm_P1.27mm" H 5950 3900 50  0001 C CNN
 F 3 "http://ww1.microchip.com/downloads/en/DeviceDoc/21733j.pdf" H 6050 4000 50  0001 C CNN
 	1    6000 3800
@@
 F 0 "U3" H 7208 2096 50  0000 L CNN
 F 1 "MCP6004" H 7208 2005 50  0000 L CNN
-F 2 "Package_DIP:DIP-14_W7.62mm" H 7200 2150 50  0001 C CNN
+F 2 "Package_SO:SOIC-16_4.55x10.3mm_P1.27mm" H 7200 2150 50  0001 C CNN
 F 3 "http://ww1.microchip.com/downloads/en/DeviceDoc/21733j.pdf" H 7300 2250 50  0001 C CNN
 	5    7250 2050

Commit message: updated resistors to 0805 on amp.sch
Parts:
- R1, R2, R3, R4, R5, R6, R7: footprint Resistor_THT:R_Axial_DIN0204_L3.6mm_D1.6mm_P5.08mm_Horizontal -> Resistor_SMD:R_0805_2012Metric_Pad1.20x1.40mm_HandSolder
Changed lines of the file:
@@
 F 0 "R6" H 5520 4096 50  0000 L CNN
 F 1 "15" H 5520 4005 50  0000 L CNN
-F 2 "Resistor_THT:R_Axial_DIN0204_L3.6mm_D1.6mm_P5.08mm_Horizontal" V 5380 4050 50  0001 C CNN
+F 2 "Resistor_SMD:R_0805_2012Metric_Pad1.20x1.40mm_HandSolder" V 5380 4050 50  0001 C CNN
 F 3 "~" H 5450 4050 50  0001 C CNN
 	1    5450 4050
@@
 F 0 "R7" V 5743 3250 50  0000 C CNN
 F 1 "15" V 5834 3250 50  0000 C CNN
-F 2 "Resistor_THT:R_Axial_DIN0204_L3.6mm_D1.6mm_P5.08mm_Horizontal" V 5880 3250 50  0001 C CNN
+F 2 "Resistor_SMD:R_0805_2012Metric_Pad1.20x1.40mm_HandSolder" V 5880 3250 50  0001 C CNN
 F 3 "~" H 5950 3250 50  0001 C CNN
 	1    5950 3250
@@
 F 0 "R4" V 5307 3700 50  0000 C CNN
 F 1 "1" V 5216 3700 50  0000 C CNN
-F 2 "Resistor_THT:R_Axial_DIN0204_L3.6mm_D1.6mm_P5.08mm_Horizontal" V 5030 3700 50  0001 C CNN
+F 2 "Resistor_SMD:R_0805_2012Metric_Pad1.20x1.40mm_HandSolder" V 5030 3700 50  0001 C CNN
 F 3 "~" H 5100 3700 50  0001 C CNN
 	1    5100 3700
@@
 F 0 "R5" V 5000 3900 50  0000 C CNN
 F 1 "1" V 4900 3900 50  0000 C CNN
-F 2 "Resistor_THT:R_Axial_DIN0204_L3.6mm_D1.6mm_P5.08mm_Horizontal" V 5030 3900 50  0001 C CNN
+F 2 "Resistor_SMD:R_0805_2012Metric_Pad1.20x1.40mm_HandSolder" V 5030 3900 50  0001 C CNN
 F 3 "~" H 5100 3900 50  0001 C CNN
 	1    5100 3900
@@
 F 0 "R1" H 3320 3546 50  0000 L CNN
 F 1 "560" H 3320 3455 50  0000 L CNN
-F 2 "Resistor_THT:R_Axial_DIN0204_L3.6mm_D1.6mm_P5.08mm_Horizontal" V 3180 3500 50  0001 C CNN
+F 2 "Resistor_SMD:R_0805_2012Metric_Pad1.20x1.40mm_HandSolder" V 3180 3500 50  0001 C CNN
 F 3 "~" H 3250 3500 50  0001 C CNN
 	1    3250 3500
@@
 F 0 "R2" H 3320 3846 50  0000 L CNN
 F 1 "300" H 3320 3755 50  0000 L CNN
-F 2 "Resistor_THT:R_Axial_DIN0204_L3.6mm_D1.6mm_P5.08mm_Horizontal" V 3180 3800 50  0001 C CNN
+F 2 "Resistor_SMD:R_0805_2012Metric_Pad1.20x1.40mm_HandSolder" V 3180 3800 50  0001 C CNN
 F 3 "~" H 3250 3800 50  0001 C CNN
 	1    3250 3800
@@
 F 0 "R3" H 3720 1796 50  0000 L CNN
 F 1 "560" H 3720 1705 50  0000 L CNN
-F 2 "Resistor_THT:R_Axial_DIN0204_L3.6mm_D1.6mm_P5.08mm_Horizontal" V 3580 1750 50  0001 C CNN
+F 2 "Resistor_SMD:R_0805_2012Metric_Pad1.20x1.40mm_HandSolder" V 3580 1750 50  0001 C CNN
 F 3 "~" H 3650 1750 50  0001 C CNN
 	1    3650 1750
