File: ampA.sch (KiCad schematic (older format))
At the start: 9 parts, among them U2 Mux, U3 MCP6004

Commit message: added mux footprint/datasheet to amp.sch
Parts:
- U2: footprint Package_DIP:DIP-16_W7.62mm -> Package_SO:SOIC-16_3.9x9.9mm_P1.27mm
Changed lines of the file:
@@
 F 0 "U2" H 3375 2515 50  0000 C CNN
 F 1 "Mux" H 3375 2424 50  0000 C CNN
-F 2 "Package_DIP:DIP-16_W7.62mm" H 3350 2050 50  0001 C CNN
-F 3 "" H 3350 2050 50  0001 C CNN
+F 2 "Package_SO:SOIC-16_3.9x9.9mm_P1.27mm" H 3350 2050 50  0001 C CNN
+F 3 "https://www.digikey.com/en/products/detail/vishay-siliconix/DG409LEDY-GE3/5995262" H 3350 2050 50  0001 C CNN
 	1    3350 2050
 	1    0    0    -1
@@
 F 0 "U2" H 5928 2221 50  0000 L CNN
 F 1 "Mux" H 5928 2130 50  0000 L CNN
-F 2 "Package_DIP:DIP-16_W7.62mm" H 5700 2100 50  0001 C CNN
-F 3 "" H 5700 2100 50  0001 C CNN
+F 2 "Package_SO:SOIC-16_3.9x9.9mm_P1.27mm" H 5700 2100 50  0001 C CNN
+F 3 "https://www.digikey.com/en/products/detail/vishay-siliconix/DG409LEDY-GE3/5995262" H 5700 2100 50  0001 C CNN
 	3    5700 2100
 	1    0    0    -1

Commit message: fixed drc errors
Parts:
- U3: footprint Package_SO:SOIC-16_4.55x10.3mm_P1.27mm -> Package_SO:SOIC-16_3.9x9.9mm_P1.27mm
Changed lines of the file:
@@
 AR Path="/601B4C0E/60198F38" Ref="#PWR043"  Part="1"
 AR Path="/601B73B7/60198F38" Ref="#PWR077"  Part="1"
-F 0 "#PWR09" H 3250 3700 50  0001 C CNN
+F 0 "#PWR077" H 3250 3700 50  0001 C CNN
 F 1 "GND" H 3255 3777 50  0000 C CNN
 F 2 "" H 3250 3950 50  0001 C CNN
@@
 AR Path="/601B4C0E/6016B854" Ref="#PWR045"  Part="1"
 AR Path="/601B73B7/6016B854" Ref="#PWR079"  Part="1"
-F 0 "#PWR011" H 5450 3950 50  0001 C CNN
+F 0 "#PWR079" H 5450 3950 50  0001 C CNN
 F 1 "GND" H 5455 4027 50  0000 C CNN
 F 2 "" H 5450 4200 50  0001 C CNN
@@
 AR Path="/601B4C0E/601899DD" Ref="#PWR047"  Part="1"
 AR Path="/601B73B7/601899DD" Ref="#PWR081"  Part="1"
-F 0 "#PWR013" H 5700 2050 50  0001 C CNN
+F 0 "#PWR081" H 5700 2050 50  0001 C CNN
 F 1 "GND" H 5705 2127 50  0000 C CNN
 F 2 "" H 5700 2300 50  0001 C CNN
@@
 AR Path="/601B4C0E/60189E9E" Ref="#PWR046"  Part="1"
 AR Path="/601B73B7/60189E9E" Ref="#PWR080"  Part="1"
-F 0 "#PWR012" H 5700 1600 50  0001 C CNN
+F 0 "#PWR080" H 5700 1600 50  0001 C CNN
 F 1 "+3.3V" H 5715 1923 50  0000 C CNN
 F 2 "" H 5700 1750 50  0001 C CNN
@@
 AR Path="/601B4C0E/60195FF1" Ref="#PWR049"  Part="1"
 AR Path="/601B73B7/60195FF1" Ref="#PWR083"  Part="1"
-F 0 "#PWR015" H 7150 2100 50  0001 C CNN
+F 0 "#PWR083" H 7150 2100 50  0001 C CNN
 F 1 "GND" H 7155 2177 50  0000 C CNN
 F 2 "" H 7150 2350 50  0001 C CNN
@@
 AR Path="/601B4C0E/60198969" Ref="#PWR048"  Part="1"
 AR Path="/601B73B7/60198969" Ref="#PWR082"  Part="1"
-F 0 "#PWR014" H 7150 1600 50  0001 C CNN
+F 0 "#PWR082" H 7150 1600 50  0001 C CNN
 F 1 "+3.3V" H 7165 1923 50  0000 C CNN
 F 2 "" H 7150 1750 50  0001 C CNN
@@
 F 0 "U3" H 6000 4167 50  0000 C CNN
 F 1 "MCP6004" H 6000 4076 50  0000 C CNN
-F 2 "Package_SO:SOIC-16_4.55x10.3mm_P1.27mm" H 5950 3900 50  0001 C CNN
+F 2 "Package_SO:SOIC-16_3.9x9.9mm_P1.27mm" H 5950 3900 50  0001 C CNN
 F 3 "http://ww1.microchip.com/downloads/en/DeviceDoc/21733j.pdf" H 6050 4000 50  0001 C CNN
 	1    6000 3800
@@
 F 0 "U3" H 7208 2096 50  0000 L CNN
 F 1 "MCP6004" H 7208 2005 50  0000 L CNN
-F 2 "Package_SO:SOIC-16_4.55x10.3mm_P1.27mm" H 7200 2150 50  0001 C CNN
+F 2 "Package_SO:SOIC-16_3.9x9.9mm_P1.27mm" H 7200 2150 50  0001 C CNN
 F 3 "http://ww1.microchip.com/downloads/en/DeviceDoc/21733j.pdf" H 7300 2250 50  0001 C CNN
 	5    7250 2050
@@
 AR Path="/601B4C0E/6019D560" Ref="#PWR042"  Part="1"
 AR Path="/601B73B7/6019D560" Ref="#PWR076"  Part="1"
-F 0 "#PWR08" H 3250 3200 50  0001 C CNN
+F 0 "#PWR076" H 3250 3200 50  0001 C CNN
 F 1 "+3.3V" H 3265 3523 50  0000 C CNN
 F 2 "" H 3250 3350 50  0001 C CNN
@@
 AR Path="/601B4C0E/60202DDC" Ref="#PWR044"  Part="1"
 AR Path="/601B73B7/60202DDC" Ref="#PWR078"  Part="1"
-F 0 "#PWR010" H 3650 1450 50  0001 C CNN
+F 0 "#PWR078" H 3650 1450 50  0001 C CNN
 F 1 "+3.3V" H 3665 1773 50  0000 C CNN
 F 2 "" H 3650 1600 50  0001 C CNN

Commit message: changed solder pads to be two separate footprints
Changed lines of the file:
@@
 AR Path="/601B4C0E/6019D565" Ref="R34"  Part="1"
 AR Path="/601B73B7/6019D565" Ref="R62"  Part="1"
-F 0 "R6" H 5520 4096 50  0000 L CNN
+F 0 "R62" H 5520 4096 50  0000 L CNN
 F 1 "15" H 5520 4005 50  0000 L CNN
 F 2 "Resistor_SMD:R_0805_2012Metric_Pad1.20x1.40mm_HandSolder" V 5380 4050 50  0001 C CNN
@@
 AR Path="/601B4C0E/60198F32" Ref="R35"  Part="1"
 AR Path="/601B73B7/60198F32" Ref="R63"  Part="1"
-F 0 "R7" V 5743 3250 50  0000 C CNN
+F 0 "R63" V 5743 3250 50  0000 C CNN
 F 1 "15" V 5834 3250 50  0000 C CNN
 F 2 "Resistor_SMD:R_0805_2012Metric_Pad1.20x1.40mm_HandSolder" V 5880 3250 50  0001 C CNN
@@
 AR Path="/601B4C0E/6017E431" Ref="R32"  Part="1"
 AR Path="/601B73B7/6017E431" Ref="R60"  Part="1"
-F 0 "R4" V 5307 3700 50  0000 C CNN
+F 0 "R60" V 5307 3700 50  0000 C CNN
 F 1 "1" V 5216 3700 50  0000 C CNN
 F 2 "Resistor_SMD:R_0805_2012Metric_Pad1.20x1.40mm_HandSolder" V 5030 3700 50  0001 C CNN
@@
 AR Path="/601B4C0E/6019D568" Ref="R33"  Part="1"
 AR Path="/601B73B7/6019D568" Ref="R61"  Part="1"
-F 0 "R5" V 5000 3900 50  0000 C CNN
+F 0 "R61" V 5000 3900 50  0000 C CNN
 F 1 "1" V 4900 3900 50  0000 C CNN
 F 2 "Resistor_SMD:R_0805_2012Metric_Pad1.20x1.40mm_HandSolder" V 5030 3900 50  0001 C CNN
@@
 AR Path="/601B4C0E/6019D55E" Ref="R29"  Part="1"
 AR Path="/601B73B7/6019D55E" Ref="R57"  Part="1"
-F 0 "R1" H 3320 3546 50  0000 L CNN
+F 0 "R57" H 3320 3546 50  0000 L CNN
 F 1 "560" H 3320 3455 50  0000 L CNN
 F 2 "Resistor_SMD:R_0805_2012Metric_Pad1.20x1.40mm_HandSolder" V 3180 3500 50  0001 C CNN
@@
 AR Path="/601B4C0E/6019D55F" Ref="R30"  Part="1"
 AR Path="/601B73B7/6019D55F" Ref="R58"  Part="1"
-F 0 "R2" H 3320 3846 50  0000 L CNN
+F 0 "R58" H 3320 3846 50  0000 L CNN
 F 1 "300" H 3320 3755 50  0000 L CNN
 F 2 "Resistor_SMD:R_0805_2012Metric_Pad1.20x1.40mm_HandSolder" V 3180 3800 50  0001 C CNN
@@
 AR Path="/601B4C0E/6016DEDC" Ref="U5"  Part="1"
 AR Path="/601B73B7/6016DEDC" Ref="U8"  Part="1"
-F 0 "U2" H 3375 2515 50  0000 C CNN
+F 0 "U8" H 3375 2515 50  0000 C CNN
 F 1 "Mux" H 3375 2424 50  0000 C CNN
 F 2 "Package_SO:SOIC-16_3.9x9.9mm_P1.27mm" H 3350 2050 50  0001 C CNN
@@
 AR Path="/601B4C0E/6016F806" Ref="U5"  Part="3"
 AR Path="/601B73B7/6016F806" Ref="U8"  Part="3"
-F 0 "U2" H 5928 2221 50  0000 L CNN
+F 0 "U8" H 5928 2221 50  0000 L CNN
 F 1 "Mux" H 5928 2130 50  0000 L CNN
 F 2 "Package_SO:SOIC-16_3.9x9.9mm_P1.27mm" H 5700 2100 50  0001 C CNN
@@
 AR Path="/601B4C0E/60189002" Ref="U6"  Part="1"
 AR Path="/601B73B7/60189002" Ref="U9"  Part="1"
-F 0 "U3" H 6000 4167 50  0000 C CNN
+F 0 "U9" H 6000 4167 50  0000 C CNN
 F 1 "MCP6004" H 6000 4076 50  0000 C CNN
 F 2 "Package_SO:SOIC-16_3.9x9.9mm_P1.27mm" H 5950 3900 50  0001 C CNN
@@
 AR Path="/601B4C0E/6018B5B8" Ref="U6"  Part="5"
 AR Path="/601B73B7/6018B5B8" Ref="U9"  Part="5"
-F 0 "U3" H 7208 2096 50  0000 L CNN
+F 0 "U9" H 7208 2096 50  0000 L CNN
 F 1 "MCP6004" H 7208 2005 50  0000 L CNN
 F 2 "Package_SO:SOIC-16_3.9x9.9mm_P1.27mm" H 7200 2150 50  0001 C CNN
@@
 AR Path="/601B4C0E/60202CFB" Ref="R31"  Part="1"
 AR Path="/601B73B7/60202CFB" Ref="R59"  Part="1"
-F 0 "R3" H 3720 1796 50  0000 L CNN
+F 0 "R59" H 3720 1796 50  0000 L CNN
 F 1 "560" H 3720 1705 50  0000 L CNN
 F 2 "Resistor_SMD:R_0805_2012Metric_Pad1.20x1.40mm_HandSolder" V 3580 1750 50  0001 C CNN

Commit message: switched over remaining rs to 0805
Changed lines of the file:
@@
 AR Path="/601B4C0E/6019D565" Ref="R34"  Part="1"
 AR Path="/601B73B7/6019D565" Ref="R62"  Part="1"
-F 0 "R62" H 5520 4096 50  0000 L CNN
+F 0 "R6" H 5520 4096 50  0000 L CNN
 F 1 "15" H 5520 4005 50  0000 L CNN
 F 2 "Resistor_SMD:R_0805_2012Metric_Pad1.20x1.40mm_HandSolder" V 5380 4050 50  0001 C CNN
@@
 AR Path="/601B4C0E/60198F32" Ref="R35"  Part="1"
 AR Path="/601B73B7/60198F32" Ref="R63"  Part="1"
-F 0 "R63" V 5743 3250 50  0000 C CNN
+F 0 "R7" V 5743 3250 50  0000 C CNN
 F 1 "15" V 5834 3250 50  0000 C CNN
 F 2 "Resistor_SMD:R_0805_2012Metric_Pad1.20x1.40mm_HandSolder" V 5880 3250 50  0001 C CNN
@@
 AR Path="/601B4C0E/6017E431" Ref="R32"  Part="1"
 AR Path="/601B73B7/6017E431" Ref="R60"  Part="1"
-F 0 "R60" V 5307 3700 50  0000 C CNN
+F 0 "R4" V 5307 3700 50  0000 C CNN
 F 1 "1" V 5216 3700 50  0000 C CNN
 F 2 "Resistor_SMD:R_0805_2012Metric_Pad1.20x1.40mm_HandSolder" V 5030 3700 50  0001 C CNN
@@
 AR Path="/601B4C0E/6019D568" Ref="R33"  Part="1"
 AR Path="/601B73B7/6019D568" Ref="R61"  Part="1"
-F 0 "R61" V 5000 3900 50  0000 C CNN
+F 0 "R5" V 5000 3900 50  0000 C CNN
 F 1 "1" V 4900 3900 50  0000 C CNN
 F 2 "Resistor_SMD:R_0805_2012Metric_Pad1.20x1.40mm_HandSolder" V 5030 3900 50  0001 C CNN
@@
 AR Path="/601B4C0E/6019D55E" Ref="R29"  Part="1"
 AR Path="/601B73B7/6019D55E" Ref="R57"  Part="1"
-F 0 "R57" H 3320 3546 50  0000 L CNN
+F 0 "R1" H 3320 3546 50  0000 L CNN
 F 1 "560" H 3320 3455 50  0000 L CNN
 F 2 "Resistor_SMD:R_0805_2012Metric_Pad1.20x1.40mm_HandSolder" V 3180 3500 50  0001 C CNN
@@
 AR Path="/601B4C0E/6019D55F" Ref="R30"  Part="1"
 AR Path="/601B73B7/6019D55F" Ref="R58"  Part="1"
-F 0 "R58" H 3320 3846 50  0000 L CNN
+F 0 "R2" H 3320 3846 50  0000 L CNN
 F 1 "300" H 3320 3755 50  0000 L CNN
 F 2 "Resistor_SMD:R_0805_2012Metric_Pad1.20x1.40mm_HandSolder" V 3180 3800 50  0001 C CNN
@@
 AR Path="/601B4C0E/60198F38" Ref="#PWR043"  Part="1"
 AR Path="/601B73B7/60198F38" Ref="#PWR077"  Part="1"
-F 0 "#PWR077" H 3250 3700 50  0001 C CNN
+F 0 "#PWR09" H 3250 3700 50  0001 C CNN
 F 1 "GND" H 3255 3777 50  0000 C CNN
 F 2 "" H 3250 3950 50  0001 C CNN
@@
 AR Path="/601B4C0E/6016B854" Ref="#PWR045"  Part="1"
 AR Path="/601B73B7/6016B854" Ref="#PWR079"  Part="1"
-F 0 "#PWR079" H 5450 3950 50  0001 C CNN
+F 0 "#PWR011" H 5450 3950 50  0001 C CNN
 F 1 "GND" H 5455 4027 50  0000 C CNN
 F 2 "" H 5450 4200 50  0001 C CNN
@@
 AR Path="/601B4C0E/601899DD" Ref="#PWR047"  Part="1"
 AR Path="/601B73B7/601899DD" Ref="#PWR081"  Part="1"
-F 0 "#PWR081" H 5700 2050 50  0001 C CNN
+F 0 "#PWR013" H 5700 2050 50  0001 C CNN
 F 1 "GND" H 5705 2127 50  0000 C CNN
 F 2 "" H 5700 2300 50  0001 C CNN
@@
 AR Path="/601B4C0E/60189E9E" Ref="#PWR046"  Part="1"
 AR Path="/601B73B7/60189E9E" Ref="#PWR080"  Part="1"
-F 0 "#PWR080" H 5700 1600 50  0001 C CNN
+F 0 "#PWR012" H 5700 1600 50  0001 C CNN
 F 1 "+3.3V" H 5715 1923 50  0000 C CNN
 F 2 "" H 5700 1750 50  0001 C CNN
@@
 AR Path="/601B4C0E/60195FF1" Ref="#PWR049"  Part="1"
 AR Path="/601B73B7/60195FF1" Ref="#PWR083"  Part="1"
-F 0 "#PWR083" H 7150 2100 50  0001 C CNN
+F 0 "#PWR015" H 7150 2100 50  0001 C CNN
 F 1 "GND" H 7155 2177 50  0000 C CNN
 F 2 "" H 7150 2350 50  0001 C CNN
@@
 AR Path="/601B4C0E/60198969" Ref="#PWR048"  Part="1"
 AR Path="/601B73B7/60198969" Ref="#PWR082"  Part="1"
-F 0 "#PWR082" H 7150 1600 50  0001 C CNN
+F 0 "#PWR014" H 7150 1600 50  0001 C CNN
 F 1 "+3.3V" H 7165 1923 50  0000 C CNN
 F 2 "" H 7150 1750 50  0001 C CNN
@@
 AR Path="/601B4C0E/6016DEDC" Ref="U5"  Part="1"
 AR Path="/601B73B7/6016DEDC" Ref="U8"  Part="1"
-F 0 "U8" H 3375 2515 50  0000 C CNN
+F 0 "U2" H 3375 2515 50  0000 C CNN
 F 1 "Mux" H 3375 2424 50  0000 C CNN
 F 2 "Package_SO:SOIC-16_3.9x9.9mm_P1.27mm" H 3350 2050 50  0001 C CNN
@@
 AR Path="/601B4C0E/6016F806" Ref="U5"  Part="3"
 AR Path="/601B73B7/6016F806" Ref="U8"  Part="3"
-F 0 "U8" H 5928 2221 50  0000 L CNN
+F 0 "U2" H 5928 2221 50  0000 L CNN
 F 1 "Mux" H 5928 2130 50  0000 L CNN
 F 2 "Package_SO:SOIC-16_3.9x9.9mm_P1.27mm" H 5700 2100 50  0001 C CNN
@@
 AR Path="/601B4C0E/60189002" Ref="U6"  Part="1"
 AR Path="/601B73B7/60189002" Ref="U9"  Part="1"
-F 0 "U9" H 6000 4167 50  0000 C CNN
+F 0 "U3" H 6000 4167 50  0000 C CNN
 F 1 "MCP6004" H 6000 4076 50  0000 C CNN
 F 2 "Package_SO:SOIC-16_3.9x9.9mm_P1.27mm" H 5950 3900 50  0001 C CNN
@@
 AR Path="/601B4C0E/6018B5B8" Ref="U6"  Part="5"
 AR Path="/601B73B7/6018B5B8" Ref="U9"  Part="5"
-F 0 "U9" H 7208 2096 50  0000 L CNN
+F 0 "U3" H 7208 2096 50  0000 L CNN
 F 1 "MCP6004" H 7208 2005 50  0000 L CNN
 F 2 "Package_SO:SOIC-16_3.9x9.9mm_P1.27mm" H 7200 2150 50  0001 C CNN
@@
 AR Path="/601B4C0E/6019D560" Ref="#PWR042"  Part="1"
 AR Path="/601B73B7/6019D560" Ref="#PWR076"  Part="1"
-F 0 "#PWR076" H 3250 3200 50  0001 C CNN
+F 0 "#PWR08" H 3250 3200 50  0001 C CNN
 F 1 "+3.3V" H 3265 3523 50  0000 C CNN
 F 2 "" H 3250 3350 50  0001 C CNN
@@
 AR Path="/601B4C0E/60202CFB" Ref="R31"  Part="1"
 AR Path="/601B73B7/60202CFB" Ref="R59"  Part="1"
-F 0 "R59" H 3720 1796 50  0000 L CNN
+F 0 "R3" H 3720 1796 50  0000 L CNN
 F 1 "560" H 3720 1705 50  0000 L CNN
 F 2 "Resistor_SMD:R_0805_2012Metric_Pad1.20x1.40mm_HandSolder" V 3580 1750 50  0001 C CNN
@@
 AR Path="/601B4C0E/60202DDC" Ref="#PWR044"  Part="1"
 AR Path="/601B73B7/60202DDC" Ref="#PWR078"  Part="1"
-F 0 "#PWR078" H 3650 1450 50  0001 C CNN
+F 0 "#PWR010" H 3650 1450 50  0001 C CNN
 F 1 "+3.3V" H 3665 1773 50  0000 C CNN
 F 2 "" H 3650 1600 50  0001 C CNN

Commit message: fixed issue with wrong amp footprint
Parts:
- U3: footprint Package_SO:SOIC-16_3.9x9.9mm_P1.27mm -> Package_SO:SOIC-14_3.9x8.7mm_P1.27mm
Changed lines of the file:
@@
 F 0 "U3" H 6000 4167 50  0000 C CNN
 F 1 "MCP6004" H 6000 4076 50  0000 C CNN
-F 2 "Package_SO:SOIC-16_3.9x9.9mm_P1.27mm" H 5950 3900 50  0001 C CNN
+F 2 "Package_SO:SOIC-14_3.9x8.7mm_P1.27mm" H 5950 3900 50  0001 C CNN
 F 3 "http://ww1.microchip.com/downloads/en/DeviceDoc/21733j.pdf" H 6050 4000 50  0001 C CNN
 	1    6000 3800
@@
 F 0 "U3" H 7208 2096 50  0000 L CNN
 F 1 "MCP6004" H 7208 2005 50  0000 L CNN
-F 2 "Package_SO:SOIC-16_3.9x9.9mm_P1.27mm" H 7200 2150 50  0001 C CNN
+F 2 "Package_SO:SOIC-14_3.9x8.7mm_P1.27mm" H 7200 2150 50  0001 C CNN
 F 3 "http://ww1.microchip.com/downloads/en/DeviceDoc/21733j.pdf" H 7300 2250 50  0001 C CNN
 	5    7250 2050

Commit message: updated sch with pico connectors
Changed lines of the file:
@@
 $Descr A4 11693 8268
 encoding utf-8
-Sheet 2 41
+Sheet 2 21
 Title ""
 Date ""
@@
 $EndComp
 $Sheet
-S 1000 1800 550  200
+S 1000 1850 550  350
 U 60194350
-F0 "sensora0" 50
+F0 "sensora" 50
 F1 "sensor.sch" 50
-F2 "Vsense" I R 1550 1900 50
+F2 "Vsense0" I R 1550 1900 50
+F3 "Vsense1" I R 1550 2000 50
+F4 "Vsense2" I R 1550 2100 50
 $EndSheet
-Wire Wire Line
-	1550 2550 2000 2550
-Text Label 2000 2550 2    50   ~ 0
+Text Label 2000 2000 2    50   ~ 0
 mux1
-$Sheet
-S 1000 2450 550  200
-U 6019B999
-F0 "sensora1" 50
-F1 "sensor.sch" 50
-F2 "Vsense" I R 1550 2550 50
-$EndSheet
-Wire Wire Line
-	1550 3200 2000 3200
-Text Label 2000 3200 2    50   ~ 0
+Text Label 2000 2100 2    50   ~ 0
 mux2
-$Sheet
-S 1000 3100 550  200
-U 6019BDB6
-F0 "sensora2" 50
-F1 "sensor.sch" 50
-F2 "Vsense" I R 1550 3200 50
-$EndSheet
 $Comp
 L power:+3.3V #PWR?
@@
 Wire Wire Line
 	3650 1900 3650 2050
+Wire Wire Line
+	1550 2000 2000 2000
+Wire Wire Line
+	1550 2100 2000 2100
 $EndSCHEMATC

Commit message: left off reworking bottom of board
Changed lines of the file:
@@
 AR Path="/601B4C0E/6019D565" Ref="R34"  Part="1"
 AR Path="/601B73B7/6019D565" Ref="R62"  Part="1"
-F 0 "R6" H 5520 4096 50  0000 L CNN
+F 0 "R62" H 5520 4096 50  0000 L CNN
 F 1 "15" H 5520 4005 50  0000 L CNN
 F 2 "Resistor_SMD:R_0805_2012Metric_Pad1.20x1.40mm_HandSolder" V 5380 4050 50  0001 C CNN
@@
 AR Path="/601B4C0E/60198F32" Ref="R35"  Part="1"
 AR Path="/601B73B7/60198F32" Ref="R63"  Part="1"
-F 0 "R7" V 5743 3250 50  0000 C CNN
+F 0 "R63" V 5743 3250 50  0000 C CNN
 F 1 "15" V 5834 3250 50  0000 C CNN
 F 2 "Resistor_SMD:R_0805_2012Metric_Pad1.20x1.40mm_HandSolder" V 5880 3250 50  0001 C CNN
@@
 AR Path="/601B4C0E/6017E431" Ref="R32"  Part="1"
 AR Path="/601B73B7/6017E431" Ref="R60"  Part="1"
-F 0 "R4" V 5307 3700 50  0000 C CNN
+F 0 "R60" V 5307 3700 50  0000 C CNN
 F 1 "1" V 5216 3700 50  0000 C CNN
 F 2 "Resistor_SMD:R_0805_2012Metric_Pad1.20x1.40mm_HandSolder" V 5030 3700 50  0001 C CNN
@@
 AR Path="/601B4C0E/6019D568" Ref="R33"  Part="1"
 AR Path="/601B73B7/6019D568" Ref="R61"  Part="1"
-F 0 "R5" V 5000 3900 50  0000 C CNN
+F 0 "R61" V 5000 3900 50  0000 C CNN
 F 1 "1" V 4900 3900 50  0000 C CNN
 F 2 "Resistor_SMD:R_0805_2012Metric_Pad1.20x1.40mm_HandSolder" V 5030 3900 50  0001 C CNN
@@
 AR Path="/601B4C0E/6019D55E" Ref="R29"  Part="1"
 AR Path="/601B73B7/6019D55E" Ref="R57"  Part="1"
-F 0 "R1" H 3320 3546 50  0000 L CNN
+F 0 "R57" H 3320 3546 50  0000 L CNN
 F 1 "560" H 3320 3455 50  0000 L CNN
 F 2 "Resistor_SMD:R_0805_2012Metric_Pad1.20x1.40mm_HandSolder" V 3180 3500 50  0001 C CNN
@@
 AR Path="/601B4C0E/6019D55F" Ref="R30"  Part="1"
 AR Path="/601B73B7/6019D55F" Ref="R58"  Part="1"
-F 0 "R2" H 3320 3846 50  0000 L CNN
+F 0 "R58" H 3320 3846 50  0000 L CNN
 F 1 "300" H 3320 3755 50  0000 L CNN
 F 2 "Resistor_SMD:R_0805_2012Metric_Pad1.20x1.40mm_HandSolder" V 3180 3800 50  0001 C CNN
@@
 AR Path="/601B4C0E/60198F38" Ref="#PWR043"  Part="1"
 AR Path="/601B73B7/60198F38" Ref="#PWR077"  Part="1"
-F 0 "#PWR09" H 3250 3700 50  0001 C CNN
+F 0 "#PWR077" H 3250 3700 50  0001 C CNN
 F 1 "GND" H 3255 3777 50  0000 C CNN
 F 2 "" H 3250 3950 50  0001 C CNN
@@
 AR Path="/601B4C0E/6016B854" Ref="#PWR045"  Part="1"
 AR Path="/601B73B7/6016B854" Ref="#PWR079"  Part="1"
-F 0 "#PWR011" H 5450 3950 50  0001 C CNN
+F 0 "#PWR079" H 5450 3950 50  0001 C CNN
 F 1 "GND" H 5455 4027 50  0000 C CNN
 F 2 "" H 5450 4200 50  0001 C CNN
@@
 AR Path="/601B4C0E/601899DD" Ref="#PWR047"  Part="1"
 AR Path="/601B73B7/601899DD" Ref="#PWR081"  Part="1"
-F 0 "#PWR013" H 5700 2050 50  0001 C CNN
+F 0 "#PWR081" H 5700 2050 50  0001 C CNN
 F 1 "GND" H 5705 2127 50  0000 C CNN
 F 2 "" H 5700 2300 50  0001 C CNN
@@
 AR Path="/601B4C0E/60189E9E" Ref="#PWR046"  Part="1"
 AR Path="/601B73B7/60189E9E" Ref="#PWR080"  Part="1"
-F 0 "#PWR012" H 5700 1600 50  0001 C CNN
+F 0 "#PWR080" H 5700 1600 50  0001 C CNN
 F 1 "+3.3V" H 5715 1923 50  0000 C CNN
 F 2 "" H 5700 1750 50  0001 C CNN
@@
 AR Path="/601B4C0E/60195FF1" Ref="#PWR049"  Part="1"
 AR Path="/601B73B7/60195FF1" Ref="#PWR083"  Part="1"
-F 0 "#PWR015" H 7150 2100 50  0001 C CNN
+F 0 "#PWR083" H 7150 2100 50  0001 C CNN
 F 1 "GND" H 7155 2177 50  0000 C CNN
 F 2 "" H 7150 2350 50  0001 C CNN
@@
 AR Path="/601B4C0E/60198969" Ref="#PWR048"  Part="1"
 AR Path="/601B73B7/60198969" Ref="#PWR082"  Part="1"
-F 0 "#PWR014" H 7150 1600 50  0001 C CNN
+F 0 "#PWR082" H 7150 1600 50  0001 C CNN
 F 1 "+3.3V" H 7165 1923 50  0000 C CNN
 F 2 "" H 7150 1750 50  0001 C CNN
@@
 AR Path="/601B4C0E/6016DEDC" Ref="U5"  Part="1"
 AR Path="/601B73B7/6016DEDC" Ref="U8"  Part="1"
-F 0 "U2" H 3375 2515 50  0000 C CNN
+F 0 "U8" H 3375 2515 50  0000 C CNN
 F 1 "Mux" H 3375 2424 50  0000 C CNN
 F 2 "Package_SO:SOIC-16_3.9x9.9mm_P1.27mm" H 3350 2050 50  0001 C CNN
@@
 AR Path="/601B4C0E/6016F806" Ref="U5"  Part="3"
 AR Path="/601B73B7/6016F806" Ref="U8"  Part="3"
-F 0 "U2" H 5928 2221 50  0000 L CNN
+F 0 "U8" H 5928 2221 50  0000 L CNN
 F 1 "Mux" H 5928 2130 50  0000 L CNN
 F 2 "Package_SO:SOIC-16_3.9x9.9mm_P1.27mm" H 5700 2100 50  0001 C CNN
@@
 AR Path="/601B4C0E/60189002" Ref="U6"  Part="1"
 AR Path="/601B73B7/60189002" Ref="U9"  Part="1"
-F 0 "U3" H 6000 4167 50  0000 C CNN
+F 0 "U9" H 6000 4167 50  0000 C CNN
 F 1 "MCP6004" H 6000 4076 50  0000 C CNN
 F 2 "Package_SO:SOIC-14_3.9x8.7mm_P1.27mm" H 5950 3900 50  0001 C CNN
@@
 AR Path="/601B4C0E/6018B5B8" Ref="U6"  Part="5"
 AR Path="/601B73B7/6018B5B8" Ref="U9"  Part="5"
-F 0 "U3" H 7208 2096 50  0000 L CNN
+F 0 "U9" H 7208 2096 50  0000 L CNN
 F 1 "MCP6004" H 7208 2005 50  0000 L CNN
 F 2 "Package_SO:SOIC-14_3.9x8.7mm_P1.27mm" H 7200 2150 50  0001 C CNN
@@
 AR Path="/601B4C0E/6019D560" Ref="#PWR042"  Part="1"
 AR Path="/601B73B7/6019D560" Ref="#PWR076"  Part="1"
-F 0 "#PWR08" H 3250 3200 50  0001 C CNN
+F 0 "#PWR076" H 3250 3200 50  0001 C CNN
 F 1 "+3.3V" H 3265 3523 50  0000 C CNN
 F 2 "" H 3250 3350 50  0001 C CNN
@@
 AR Path="/601B4C0E/60202CFB" Ref="R31"  Part="1"
 AR Path="/601B73B7/60202CFB" Ref="R59"  Part="1"
-F 0 "R3" H 3720 1796 50  0000 L CNN
+F 0 "R59" H 3720 1796 50  0000 L CNN
 F 1 "560" H 3720 1705 50  0000 L CNN
 F 2 "Resistor_SMD:R_0805_2012Metric_Pad1.20x1.40mm_HandSolder" V 3580 1750 50  0001 C CNN
@@
 AR Path="/601B4C0E/60202DDC" Ref="#PWR044"  Part="1"
 AR Path="/601B73B7/60202DDC" Ref="#PWR078"  Part="1"
-F 0 "#PWR010" H 3650 1450 50  0001 C CNN
+F 0 "#PWR078" H 3650 1450 50  0001 C CNN
 F 1 "+3.3V" H 3665 1773 50  0000 C CNN
 F 2 "" H 3650 1600 50  0001 C CNN
