File: ampB.sch (KiCad schematic (older format))
At the start: 9 parts, among them U2 Mux, U3 MCP6004

Commit message: reverted back to screw terminals
Changed lines of the file:
@@
 AR Path="/601B4C11/6019E3A5" Ref="R41"  Part="1"
 AR Path="/601B73BA/6019E3A5" Ref="R69"  Part="1"
-F 0 "R13" H 5520 4096 50  0000 L CNN
+F 0 "R69" H 5520 4096 50  0000 L CNN
 F 1 "15" H 5520 4005 50  0000 L CNN
 F 2 "Resistor_SMD:R_0805_2012Metric_Pad1.20x1.40mm_HandSolder" V 5380 4050 50  0001 C CNN
@@
 AR Path="/601B4C11/6017E430" Ref="R42"  Part="1"
 AR Path="/601B73BA/6017E430" Ref="R70"  Part="1"
-F 0 "R14" V 5743 3250 50  0000 C CNN
+F 0 "R70" V 5743 3250 50  0000 C CNN
 F 1 "15" V 5834 3250 50  0000 C CNN
 F 2 "Resistor_SMD:R_0805_2012Metric_Pad1.20x1.40mm_HandSolder" V 5880 3250 50  0001 C CNN
@@
 AR Path="/601B4C11/60198F33" Ref="R39"  Part="1"
 AR Path="/601B73BA/60198F33" Ref="R67"  Part="1"
-F 0 "R11" V 5307 3700 50  0000 C CNN
+F 0 "R67" V 5307 3700 50  0000 C CNN
 F 1 "1" V 5216 3700 50  0000 C CNN
 F 2 "Resistor_SMD:R_0805_2012Metric_Pad1.20x1.40mm_HandSolder" V 5030 3700 50  0001 C CNN
@@
 AR Path="/601B4C11/6017E432" Ref="R40"  Part="1"
 AR Path="/601B73BA/6017E432" Ref="R68"  Part="1"
-F 0 "R12" V 5000 3900 50  0000 C CNN
+F 0 "R68" V 5000 3900 50  0000 C CNN
 F 1 "1" V 4900 3900 50  0000 C CNN
 F 2 "Resistor_SMD:R_0805_2012Metric_Pad1.20x1.40mm_HandSolder" V 5030 3900 50  0001 C CNN
@@
 AR Path="/601B4C11/60198F35" Ref="R36"  Part="1"
 AR Path="/601B73BA/60198F35" Ref="R64"  Part="1"
-F 0 "R8" H 3320 3546 50  0000 L CNN
+F 0 "R64" H 3320 3546 50  0000 L CNN
 F 1 "560" H 3320 3455 50  0000 L CNN
 F 2 "Resistor_SMD:R_0805_2012Metric_Pad1.20x1.40mm_HandSolder" V 3180 3500 50  0001 C CNN
@@
 AR Path="/601B4C11/6019E3B4" Ref="R37"  Part="1"
 AR Path="/601B73BA/6019E3B4" Ref="R65"  Part="1"
-F 0 "R9" H 3320 3846 50  0000 L CNN
+F 0 "R65" H 3320 3846 50  0000 L CNN
 F 1 "300" H 3320 3755 50  0000 L CNN
 F 2 "Resistor_SMD:R_0805_2012Metric_Pad1.20x1.40mm_HandSolder" V 3180 3800 50  0001 C CNN
@@
 AR Path="/601B4C11/6019E3B5" Ref="#PWR053"  Part="1"
 AR Path="/601B73BA/6019E3B5" Ref="#PWR087"  Part="1"
-F 0 "#PWR019" H 3250 3200 50  0001 C CNN
+F 0 "#PWR087" H 3250 3200 50  0001 C CNN
 F 1 "+3.3V" H 3265 3523 50  0000 C CNN
 F 2 "" H 3250 3350 50  0001 C CNN
@@
 AR Path="/601B4C11/6017E436" Ref="#PWR054"  Part="1"
 AR Path="/601B73BA/6017E436" Ref="#PWR088"  Part="1"
-F 0 "#PWR020" H 3250 3700 50  0001 C CNN
+F 0 "#PWR088" H 3250 3700 50  0001 C CNN
 F 1 "GND" H 3255 3777 50  0000 C CNN
 F 2 "" H 3250 3950 50  0001 C CNN
@@
 AR Path="/601B4C11/6019E3AC" Ref="#PWR056"  Part="1"
 AR Path="/601B73BA/6019E3AC" Ref="#PWR090"  Part="1"
-F 0 "#PWR022" H 5450 3950 50  0001 C CNN
+F 0 "#PWR090" H 5450 3950 50  0001 C CNN
 F 1 "GND" H 5455 4027 50  0000 C CNN
 F 2 "" H 5450 4200 50  0001 C CNN
@@
 AR Path="/601B4C11/6017859B" Ref="U5"  Part="2"
 AR Path="/601B73BA/6017859B" Ref="U8"  Part="2"
-F 0 "U2" H 3375 2515 50  0000 C CNN
+F 0 "U8" H 3375 2515 50  0000 C CNN
 F 1 "Mux" H 3375 2424 50  0000 C CNN
 F 2 "Package_SO:SOIC-16_3.9x9.9mm_P1.27mm" H 3350 2050 50  0001 C CNN
@@
 AR Path="/601B4C11/6018C8DB" Ref="U6"  Part="2"
 AR Path="/601B73BA/6018C8DB" Ref="U9"  Part="2"
-F 0 "U3" H 6000 4167 50  0000 C CNN
+F 0 "U9" H 6000 4167 50  0000 C CNN
 F 1 "MCP6004" H 6000 4076 50  0000 C CNN
 F 2 "Package_SO:SOIC-14_3.9x8.7mm_P1.27mm" H 5950 3900 50  0001 C CNN
@@
 AR Path="/601B4C11/602069C8" Ref="R38"  Part="1"
 AR Path="/601B73BA/602069C8" Ref="R66"  Part="1"
-F 0 "R10" H 3720 1946 50  0000 L CNN
+F 0 "R66" H 3720 1946 50  0000 L CNN
 F 1 "560" H 3720 1855 50  0000 L CNN
 F 2 "Resistor_SMD:R_0805_2012Metric_Pad1.20x1.40mm_HandSolder" V 3580 1900 50  0001 C CNN
@@
 AR Path="/601B4C11/60206B01" Ref="#PWR055"  Part="1"
 AR Path="/601B73BA/60206B01" Ref="#PWR089"  Part="1"
-F 0 "#PWR021" H 3650 1600 50  0001 C CNN
+F 0 "#PWR089" H 3650 1600 50  0001 C CNN
 F 1 "+3.3V" H 3665 1923 50  0000 C CNN
 F 2 "" H 3650 1750 50  0001 C CNN

Commit message: updated sch with pico connectors
Changed lines of the file:
@@
 $Descr A4 11693 8268
 encoding utf-8
-Sheet 6 41
+Sheet 4 21
 Title ""
 Date ""
@@
 AR Path="/601B4C11/6019E3A5" Ref="R41"  Part="1"
 AR Path="/601B73BA/6019E3A5" Ref="R69"  Part="1"
-F 0 "R69" H 5520 4096 50  0000 L CNN
+F 0 "R13" H 5520 4096 50  0000 L CNN
 F 1 "15" H 5520 4005 50  0000 L CNN
 F 2 "Resistor_SMD:R_0805_2012Metric_Pad1.20x1.40mm_HandSolder" V 5380 4050 50  0001 C CNN
@@
 AR Path="/601B4C11/6017E430" Ref="R42"  Part="1"
 AR Path="/601B73BA/6017E430" Ref="R70"  Part="1"
-F 0 "R70" V 5743 3250 50  0000 C CNN
+F 0 "R14" V 5743 3250 50  0000 C CNN
 F 1 "15" V 5834 3250 50  0000 C CNN
 F 2 "Resistor_SMD:R_0805_2012Metric_Pad1.20x1.40mm_HandSolder" V 5880 3250 50  0001 C CNN
@@
 AR Path="/601B4C11/60198F33" Ref="R39"  Part="1"
 AR Path="/601B73BA/60198F33" Ref="R67"  Part="1"
-F 0 "R67" V 5307 3700 50  0000 C CNN
+F 0 "R11" V 5307 3700 50  0000 C CNN
 F 1 "1" V 5216 3700 50  0000 C CNN
 F 2 "Resistor_SMD:R_0805_2012Metric_Pad1.20x1.40mm_HandSolder" V 5030 3700 50  0001 C CNN
@@
 AR Path="/601B4C11/6017E432" Ref="R40"  Part="1"
 AR Path="/601B73BA/6017E432" Ref="R68"  Part="1"
-F 0 "R68" V 5000 3900 50  0000 C CNN
+F 0 "R12" V 5000 3900 50  0000 C CNN
 F 1 "1" V 4900 3900 50  0000 C CNN
 F 2 "Resistor_SMD:R_0805_2012Metric_Pad1.20x1.40mm_HandSolder" V 5030 3900 50  0001 C CNN
@@
 AR Path="/601B4C11/60198F35" Ref="R36"  Part="1"
 AR Path="/601B73BA/60198F35" Ref="R64"  Part="1"
-F 0 "R64" H 3320 3546 50  0000 L CNN
+F 0 "R8" H 3320 3546 50  0000 L CNN
 F 1 "560" H 3320 3455 50  0000 L CNN
 F 2 "Resistor_SMD:R_0805_2012Metric_Pad1.20x1.40mm_HandSolder" V 3180 3500 50  0001 C CNN
@@
 AR Path="/601B4C11/6019E3B4" Ref="R37"  Part="1"
 AR Path="/601B73BA/6019E3B4" Ref="R65"  Part="1"
-F 0 "R65" H 3320 3846 50  0000 L CNN
+F 0 "R9" H 3320 3846 50  0000 L CNN
 F 1 "300" H 3320 3755 50  0000 L CNN
 F 2 "Resistor_SMD:R_0805_2012Metric_Pad1.20x1.40mm_HandSolder" V 3180 3800 50  0001 C CNN
@@
 AR Path="/601B4C11/6019E3B5" Ref="#PWR053"  Part="1"
 AR Path="/601B73BA/6019E3B5" Ref="#PWR087"  Part="1"
-F 0 "#PWR087" H 3250 3200 50  0001 C CNN
+F 0 "#PWR019" H 3250 3200 50  0001 C CNN
 F 1 "+3.3V" H 3265 3523 50  0000 C CNN
 F 2 "" H 3250 3350 50  0001 C CNN
@@
 AR Path="/601B4C11/6017E436" Ref="#PWR054"  Part="1"
 AR Path="/601B73BA/6017E436" Ref="#PWR088"  Part="1"
-F 0 "#PWR088" H 3250 3700 50  0001 C CNN
+F 0 "#PWR020" H 3250 3700 50  0001 C CNN
 F 1 "GND" H 3255 3777 50  0000 C CNN
 F 2 "" H 3250 3950 50  0001 C CNN
@@
 AR Path="/601B4C11/6019E3AC" Ref="#PWR056"  Part="1"
 AR Path="/601B73BA/6019E3AC" Ref="#PWR090"  Part="1"
-F 0 "#PWR090" H 5450 3950 50  0001 C CNN
+F 0 "#PWR022" H 5450 3950 50  0001 C CNN
 F 1 "GND" H 5455 4027 50  0000 C CNN
 F 2 "" H 5450 4200 50  0001 C CNN
@@
 AR Path="/601B4C11/6017859B" Ref="U5"  Part="2"
 AR Path="/601B73BA/6017859B" Ref="U8"  Part="2"
-F 0 "U8" H 3375 2515 50  0000 C CNN
+F 0 "U2" H 3375 2515 50  0000 C CNN
 F 1 "Mux" H 3375 2424 50  0000 C CNN
 F 2 "Package_SO:SOIC-16_3.9x9.9mm_P1.27mm" H 3350 2050 50  0001 C CNN
@@
 AR Path="/601B4C11/6018C8DB" Ref="U6"  Part="2"
 AR Path="/601B73BA/6018C8DB" Ref="U9"  Part="2"
-F 0 "U9" H 6000 4167 50  0000 C CNN
+F 0 "U3" H 6000 4167 50  0000 C CNN
 F 1 "MCP6004" H 6000 4076 50  0000 C CNN
 F 2 "Package_SO:SOIC-14_3.9x8.7mm_P1.27mm" H 5950 3900 50  0001 C CNN
@@
 mux0
 $Sheet
-S 1100 1800 550  200
+S 1100 1800 550  400
 U 601A1EA6
 F0 "sensorb0" 50
 F1 "sensor.sch" 50
-F2 "Vsense" I R 1650 1900 50
-$EndSheet
-Wire Wire Line
-	1650 2550 2100 2550
-Text Label 2100 2550 2    50   ~ 0
-mux1
-$Sheet
-S 1100 2450 550  200
-U 601A1EAB
-F0 "sensorb1" 50
-F1 "sensor.sch" 50
-F2 "Vsense" I R 1650 2550 50
-$EndSheet
-Wire Wire Line
-	1650 3200 2100 3200
-Text Label 2100 3200 2    50   ~ 0
-mux2
-$Sheet
-S 1100 3100 550  200
-U 601A1EB0
-F0 "sensorb2" 50
-F1 "sensor.sch" 50
-F2 "Vsense" I R 1650 3200 50
+F2 "Vsense0" I R 1650 1900 50
+F3 "Vsense1" I R 1650 2000 50
+F4 "Vsense2" I R 1650 2100 50
 $EndSheet
 $Comp
@@
 AR Path="/601B4C11/602069C8" Ref="R38"  Part="1"
 AR Path="/601B73BA/602069C8" Ref="R66"  Part="1"
-F 0 "R66" H 3720 1946 50  0000 L CNN
+F 0 "R10" H 3720 1946 50  0000 L CNN
 F 1 "560" H 3720 1855 50  0000 L CNN
 F 2 "Resistor_SMD:R_0805_2012Metric_Pad1.20x1.40mm_HandSolder" V 3580 1900 50  0001 C CNN
@@
 AR Path="/601B4C11/60206B01" Ref="#PWR055"  Part="1"
 AR Path="/601B73BA/60206B01" Ref="#PWR089"  Part="1"
-F 0 "#PWR089" H 3650 1600 50  0001 C CNN
+F 0 "#PWR021" H 3650 1600 50  0001 C CNN
 F 1 "+3.3V" H 3665 1923 50  0000 C CNN
 F 2 "" H 3650 1750 50  0001 C CNN
@@
 	1    0    0    -1
 $EndComp
+Text Label 2100 2100 2    50   ~ 0
+mux2
+Text Label 2100 2000 2    50   ~ 0
+mux1
+Wire Wire Line
+	1650 2100 2100 2100
+Wire Wire Line
+	2100 2000 1650 2000
 $EndSCHEMATC

Commit message: left off reworking bottom of board
Changed lines of the file:
@@
 AR Path="/601B4C11/6019E3A5" Ref="R41"  Part="1"
 AR Path="/601B73BA/6019E3A5" Ref="R69"  Part="1"
-F 0 "R13" H 5520 4096 50  0000 L CNN
+F 0 "R69" H 5520 4096 50  0000 L CNN
 F 1 "15" H 5520 4005 50  0000 L CNN
 F 2 "Resistor_SMD:R_0805_2012Metric_Pad1.20x1.40mm_HandSolder" V 5380 4050 50  0001 C CNN
@@
 AR Path="/601B4C11/6017E430" Ref="R42"  Part="1"
 AR Path="/601B73BA/6017E430" Ref="R70"  Part="1"
-F 0 "R14" V 5743 3250 50  0000 C CNN
+F 0 "R70" V 5743 3250 50  0000 C CNN
 F 1 "15" V 5834 3250 50  0000 C CNN
 F 2 "Resistor_SMD:R_0805_2012Metric_Pad1.20x1.40mm_HandSolder" V 5880 3250 50  0001 C CNN
@@
 AR Path="/601B4C11/60198F33" Ref="R39"  Part="1"
 AR Path="/601B73BA/60198F33" Ref="R67"  Part="1"
-F 0 "R11" V 5307 3700 50  0000 C CNN
+F 0 "R67" V 5307 3700 50  0000 C CNN
 F 1 "1" V 5216 3700 50  0000 C CNN
 F 2 "Resistor_SMD:R_0805_2012Metric_Pad1.20x1.40mm_HandSolder" V 5030 3700 50  0001 C CNN
@@
 AR Path="/601B4C11/6017E432" Ref="R40"  Part="1"
 AR Path="/601B73BA/6017E432" Ref="R68"  Part="1"
-F 0 "R12" V 5000 3900 50  0000 C CNN
+F 0 "R68" V 5000 3900 50  0000 C CNN
 F 1 "1" V 4900 3900 50  0000 C CNN
 F 2 "Resistor_SMD:R_0805_2012Metric_Pad1.20x1.40mm_HandSolder" V 5030 3900 50  0001 C CNN
@@
 AR Path="/601B4C11/60198F35" Ref="R36"  Part="1"
 AR Path="/601B73BA/60198F35" Ref="R64"  Part="1"
-F 0 "R8" H 3320 3546 50  0000 L CNN
+F 0 "R64" H 3320 3546 50  0000 L CNN
 F 1 "560" H 3320 3455 50  0000 L CNN
 F 2 "Resistor_SMD:R_0805_2012Metric_Pad1.20x1.40mm_HandSolder" V 3180 3500 50  0001 C CNN
@@
 AR Path="/601B4C11/6019E3B4" Ref="R37"  Part="1"
 AR Path="/601B73BA/6019E3B4" Ref="R65"  Part="1"
-F 0 "R9" H 3320 3846 50  0000 L CNN
+F 0 "R65" H 3320 3846 50  0000 L CNN
 F 1 "300" H 3320 3755 50  0000 L CNN
 F 2 "Resistor_SMD:R_0805_2012Metric_Pad1.20x1.40mm_HandSolder" V 3180 3800 50  0001 C CNN
@@
 AR Path="/601B4C11/6019E3B5" Ref="#PWR053"  Part="1"
 AR Path="/601B73BA/6019E3B5" Ref="#PWR087"  Part="1"
-F 0 "#PWR019" H 3250 3200 50  0001 C CNN
+F 0 "#PWR087" H 3250 3200 50  0001 C CNN
 F 1 "+3.3V" H 3265 3523 50  0000 C CNN
 F 2 "" H 3250 3350 50  0001 C CNN
@@
 AR Path="/601B4C11/6017E436" Ref="#PWR054"  Part="1"
 AR Path="/601B73BA/6017E436" Ref="#PWR088"  Part="1"
-F 0 "#PWR020" H 3250 3700 50  0001 C CNN
+F 0 "#PWR088" H 3250 3700 50  0001 C CNN
 F 1 "GND" H 3255 3777 50  0000 C CNN
 F 2 "" H 3250 3950 50  0001 C CNN
@@
 AR Path="/601B4C11/6019E3AC" Ref="#PWR056"  Part="1"
 AR Path="/601B73BA/6019E3AC" Ref="#PWR090"  Part="1"
-F 0 "#PWR022" H 5450 3950 50  0001 C CNN
+F 0 "#PWR090" H 5450 3950 50  0001 C CNN
 F 1 "GND" H 5455 4027 50  0000 C CNN
 F 2 "" H 5450 4200 50  0001 C CNN
@@
 AR Path="/601B4C11/6017859B" Ref="U5"  Part="2"
 AR Path="/601B73BA/6017859B" Ref="U8"  Part="2"
-F 0 "U2" H 3375 2515 50  0000 C CNN
+F 0 "U8" H 3375 2515 50  0000 C CNN
 F 1 "Mux" H 3375 2424 50  0000 C CNN
 F 2 "Package_SO:SOIC-16_3.9x9.9mm_P1.27mm" H 3350 2050 50  0001 C CNN
@@
 AR Path="/601B4C11/6018C8DB" Ref="U6"  Part="2"
 AR Path="/601B73BA/6018C8DB" Ref="U9"  Part="2"
-F 0 "U3" H 6000 4167 50  0000 C CNN
+F 0 "U9" H 6000 4167 50  0000 C CNN
 F 1 "MCP6004" H 6000 4076 50  0000 C CNN
 F 2 "Package_SO:SOIC-14_3.9x8.7mm_P1.27mm" H 5950 3900 50  0001 C CNN
@@
 AR Path="/601B4C11/602069C8" Ref="R38"  Part="1"
 AR Path="/601B73BA/602069C8" Ref="R66"  Part="1"
-F 0 "R10" H 3720 1946 50  0000 L CNN
+F 0 "R66" H 3720 1946 50  0000 L CNN
 F 1 "560" H 3720 1855 50  0000 L CNN
 F 2 "Resistor_SMD:R_0805_2012Metric_Pad1.20x1.40mm_HandSolder" V 3580 1900 50  0001 C CNN
@@
 AR Path="/601B4C11/60206B01" Ref="#PWR055"  Part="1"
 AR Path="/601B73BA/60206B01" Ref="#PWR089"  Part="1"
-F 0 "#PWR021" H 3650 1600 50  0001 C CNN
+F 0 "#PWR089" H 3650 1600 50  0001 C CNN
 F 1 "+3.3V" H 3665 1923 50  0000 C CNN
 F 2 "" H 3650 1750 50  0001 C CNN
