File: sensor.sch (KiCad schematic (older format))
At the start: 1 part, among them J1 Conn_01x06_Female

Commit message: left off with esp32 needing integration
Changed lines of the file:
@@
 AR Path="/601B73B7/60194350/60B45C6C" Ref="J9"  Part="1"
 AR Path="/601B73BA/601A1EA6/60B45C6C" Ref="J10"  Part="1"
-F 0 "J1" H 4892 4285 50  0000 C CNN
+F 0 "J10" H 4892 4285 50  0000 C CNN
 F 1 "Conn_01x06_Female" H 4892 4194 50  0000 C CNN
 F 2 "Connector_Molex:Molex_PicoBlade_53047-0610_1x06_P1.25mm_Vertical" H 5000 3900 50  0001 C CNN
